File: misc_designs/padaukprog.brd (EAGLE design)
At the start: 100 x 100 mm, 321 parts, among them IC1 LM358D, IC11 LAN8720A, IC15 TPS62063, IC4 4051D, IC5 4051D, IC6 IC_DIL16-SOIC-16, J1 JUMPER_SOLDER_1X2, J2 JUMPER_SOLDER_1X2, J3 JST-PH 2mm, J5 AVR_SPI_PRG_6NS, J6 JST-PH 2mm, J7 CON-HIROSE-COAXIAL-U.FL, M1 XT1861B, M2 XT1861B, M3 XT1861B, P1 B3B-PH-K, P2 B3B-PH-K, Q1 BSS84, Q10 BSS84, Q11 BSS84, Q12 CRISTAL-3225, Q13 CRISTAL-3225, Q2 8MHz, Q3 BSS84, Q4 BSS123, Q5 25MHz, Q6 FDN338, Q7 8MHz, Q8 BSS84, Q9 BSS84, T2 Hanrun HR917550A, U1 MIC550X, U2 STM32F107RCT6, U3 ESP-WROOM-32, U4 ATTINY24A-SSU

Commit message: Final routed
Parts:
- removed C83: (no value), GadgetFactory:0805
- removed C84, C85, C86, C87: 15pF, GadgetFactory:0402
- removed C93, C94, C95: 100nF, GadgetFactory:0603
- removed C96: 2.2uF, GadgetFactory:0805
- removed C97: 1uF, GadgetFactory:0603
- removed C98: 1nF, GadgetFactory:0603
- removed C99: 100nF/DNP, GadgetFactory:0603
- removed H8: MOUNT-PAD-ROUND3.2, holes:3,2-PAD
- removed IC11: LAN8720A, sigedi-footprints:QFN24_4MM_X_4MM
- removed IC15: TPS62063, alvie:WSON8-2.1X2.1
- removed J7: CON-HIROSE-COAXIAL-U.FL, m-pad-2.1:CON-U.FL
- removed L15: (no value), GadgetFactory:0402
- removed L16: 600R, GadgetFactory:0805
- removed LED7, LED8: LG L29K-G2J1-24, dp_devices:LED-603
- removed Q12, Q13: CRISTAL-3225, alvie:CRYSTAL-3225
- removed R84, R85, R86: 49R9, GadgetFactory:0603
- removed R87: 10K, GadgetFactory:0603
- removed SV1: MA13-2W, alvie:MA13-2W
- removed U$31, U$32, U$33: PIN-1X4, alvie:PIN-1X4
- added H6: MOUNT-PAD-ROUND3.2, holes:3,2-PAD
- added IC3: IC_DIL16-SOIC-16, dp_devices:SOIC-16
- added IC7: 4051D, 40xx:SO16
- added IC8, U$20: PFS154-S16, alvie:SOIC16-N
- added IC9: MIC550X, alvie:SOT23-5L
- added JP12, JP13, U$21, U$23: PIN-1X8, alvie:PIN-1X8
- added U$18: PIN-1X10, alvie:PIN-1X10
- added U$19: STM32F030F4P6, alvie:TSSOP20
- added U$22: PIN-1X4, alvie:PIN-1X4
- added X1, X2: FH12-40S-0.5SH, con-hirose:FH12-40S-0.5SH
- C1: value 22uF 16V -> 100nF 6.3V; device GadgetFactory:0805 -> GadgetFactory:0603
- C11, C29, C8: value 100nF 50V -> 100nF
- C12: value 22uF 50V -> 10uF; device GadgetFactory:0805 -> GadgetFactory:0603
- C13: value 22uF 50V -> 2.2uF 50V
- C14: value 100nF -> 2.2uF
- C15, C45: value 100nF 6.3V -> 100nF
- C16: value 20pF 6.3V -> 2.2uF; device GadgetFactory:0603 -> GadgetFactory:0805
- C17: value 20pF 6.3V -> 10uF
- C18: value 100nF 6.3V -> 10uF
- C19: value 100nF 6.3V -> 16pF 6.3V
- C2: value 100nF -> 100nF 6.3V
- C20: value 1uF -> 16pF 6.3V
- C21: value 100nF 50V -> 1uF
- C22, C27, C7: value 100nF 50V -> 100nF 6.3V
- C23: value 10uF -> 1nF; device GadgetFactory:0805 -> GadgetFactory:0603
- C24: value 22uF -> 100nF 6.3V; device GadgetFactory:0805 -> GadgetFactory:0603
- C25: value 10uF 6.3V -> 100nF 50V
- C26: value 100nF 6.3V -> 100nF 50V
- C28: value 10uF 6.3V -> 100nF/DNP
- C3: value 2.2uF -> 100nF 6.3V
- C30: value 10uF 6.3V -> 100nF
- C31: value 100nF 6.3V -> 20pF 6.3V
- C32: value 22uF 16V -> 20pF 6.3V; device GadgetFactory:0805 -> GadgetFactory:0603
- C33: value 10uF -> 100nF
- C34, C76: value 1uF -> 100nF
- C36, C61: value 100nF -> 1uF
- C37: value 1uF -> 10uF; device GadgetFactory:0603 -> GadgetFactory:0805
- C38: value 16pF 6.3V -> 10uF
- C39: value 16pF 6.3V -> (none); device GadgetFactory:0603 -> GadgetFactory:0805
- C4: value 10uF -> 100nF 6.3V
- C40: value 100nF 6.3V -> 22uF; device GadgetFactory:0603 -> GadgetFactory:0805
- C41: value 100nF 6.3V -> 22uF 16V; device GadgetFactory:0603 -> GadgetFactory:0805
- C42: value 100nF 6.3V -> (none); device GadgetFactory:0603 -> GadgetFactory:0805
- C43: value 100nF 6.3V -> 10uF 6.3V
- C44: value 10uF -> 22uF 16V; device GadgetFactory:0603 -> GadgetFactory:0805
- C46: value 10uF -> 1uF
- C47: value 20pF 6.3V -> 100nF 6.3V
- C48: value 10uF -> 10uF; device GadgetFactory:0805 -> GadgetFactory:0603
- C49: value 10uF -> 10uF 6.3V; device GadgetFactory:0805 -> GadgetFactory:0603
- C5: value 100nF 50V -> 22uF 16V; device GadgetFactory:0603 -> GadgetFactory:0805
- C51: value 10nF -> 10uF; device GadgetFactory:0603 -> GadgetFactory:0805
- C52: value 20pF 6.3V -> 10uF 6.3V
- C53, C57, C60: value 100nF -> 100nF 50V
- C55: value 10uF -> (none)
- C56: value 10nF -> 100nF 6.3V
- C58, C59: value 100nF -> 22uF 50V; device GadgetFactory:0603 -> GadgetFactory:0805
- C62: value (none) -> 10uF; device GadgetFactory:0603 -> GadgetFactory:0805
- C63: value (none) -> 100nF 50V
- C64: value (none) -> 100nF
- C65: value (none) -> 10nF; device GadgetFactory:0805 -> GadgetFactory:0603
- C66: value 22uF 16V -> 100nF 50V; device GadgetFactory:0805 -> GadgetFactory:0603
- C67: value 10uF -> (none); device GadgetFactory:0603 -> GadgetFactory:0805
- C69: value (none) -> 100nF; device GadgetFactory:0805 -> GadgetFactory:0603
- C70, C73, C77, C80: device GadgetFactory:0402 -> GadgetFactory:0603
- C71, C74: value (none) -> 100nF; device GadgetFactory:0402 -> GadgetFactory:0603
- C72: device GadgetFactory:0402 -> GadgetFactory:0805
- C75: value 100nF -> (none)
- C78: value 100nF -> 10uF; device GadgetFactory:0402 -> GadgetFactory:0805
- C79: value 220pF -> 10nF; device GadgetFactory:0402 -> GadgetFactory:0603
- C81: value 100nF -> 20pF 6.3V; device GadgetFactory:0402 -> GadgetFactory:0603
- C82: value 1uF -> 20pF 6.3V
- C9: value 2.2uF 50V -> 100nF 50V; device GadgetFactory:0805 -> GadgetFactory:0603
- D1: value RB521S-30 -> 1N4148W; device GadgetFactory:SOD523 -> alvie:SOD-123
- D2: value RB521S-30 -> 2SS100L-W; device GadgetFactory:SOD523 -> dp_devices:SOD-123
- D3: value 2SS100L-W -> RB521S-30; device dp_devices:SOD-123 -> GadgetFactory:SOD523
- D4: value 1N4148W -> RB521S-30; device alvie:SOD-123 -> GadgetFactory:SOD523
- IC1: value LM358D -> LAN8720A; device linear:SO08 -> sigedi-footprints:QFN24_4MM_X_4MM
- IC2: value (none) -> LM358D; device ic-package:DIL16 -> linear:SO08
- IC4: value 4051D -> TPS62063; device 40xx:SO16 -> alvie:WSON8-2.1X2.1
- IC5: value 4051D -> (none); device 40xx:SO16 -> ic-package:DIL16
- IC6: value IC_DIL16-SOIC-16 -> 4051D; device dp_devices:SOIC-16 -> 40xx:SO16
- J1: value JUMPER_SOLDER_1X2 -> JST-PH 2mm; device dp_devices:JUMPER_SOLDER_1X2 -> SparkFun-Connectors:JST-2-PTH@1
- J3: value JST-PH 2mm -> (none); device SparkFun-Connectors:JST-2-PTH@1 -> GadgetFactory:SPC4078-NOSLOT
- J4: value (none) -> JST-PH 2mm; device GadgetFactory:SPC4078-NOSLOT -> SparkFun-Connectors:JST-2-PTH@1
- J5: value AVR_SPI_PRG_6NS -> JUMPER_SOLDER_1X2; device SparkFun-Connectors:2X3-NS -> dp_devices:JUMPER_SOLDER_1X2
- J6: value JST-PH 2mm -> AVR_SPI_PRG_6NS; device SparkFun-Connectors:JST-2-PTH@1 -> SparkFun-Connectors:2X3-NS
- JP10: value PIN-1X8 -> VBat +; device alvie:PIN-1X8 -> alvie:PIN-1X2
- JP11: value PIN-1X2 -> Pedal
- JP3: value PIN-1X3 -> PIN-1X2; device alvie:PIN-1X3 -> alvie:PIN-1X2
- JP4: value PIN-1X2 -> PIN-1X3; device alvie:PIN-1X2 -> alvie:PIN-1X3
- JP6: value VBat + -> PIN-1X2
- JP8: value PIN-1X8 -> PIN-1X2; device alvie:PIN-1X8 -> alvie:PIN-1X2
- JP9: value Pedal -> PIN-1X2
- L1: value 10uH -> 10mH
- L10: value 600R -> DFE252012F; device GadgetFactory:0805 -> alvie:L2520
- L11: value DFE252012F -> 600R; device alvie:L2520 -> GadgetFactory:0805
- L13: value 10uH -> DFE252012F; device GadgetFactory:0805 -> alvie:L2520
- L14: value (none) -> 600R; device GadgetFactory:0402 -> GadgetFactory:0805
- L2: value DFE252012F -> 10uH; device alvie:L2520 -> GadgetFactory:0805
- L3: value (none) -> 10uH
- L6: value 10uH -> (none)
- L8: value 10mH -> 10uH
- L9: value 600R -> 10uH
- Q11: value BSS84 -> 8MHz; device transistor-small-signal:SOT23 -> crystal:HC49U-V
- Q2, Q7: value 8MHz -> BSS84; device crystal:HC49U-V -> transistor-small-signal:SOT23
- Q4: value BSS123 -> 25MHz; device transistor-small-signal:SOT23 -> crystal:HC49U-V
- Q5: value 25MHz -> BSS84; device crystal:HC49U-V -> transistor-small-signal:SOT23
- Q6: value FDN338 -> 8MHz; device transistor-power:SUPER-SOT3 -> crystal:HC49U-V
- Q8: value BSS84 -> BSS123
- Q9: value BSS84 -> FDN338; device transistor-small-signal:SOT23 -> transistor-power:SUPER-SOT3
- R1: value 2K2 -> 470K
- R10, R38, R8, R9: value 10K -> 2K2
- R11, R36: value 20R -> 10K
- R13: value 0R/DNP -> 330R
- R14: value 100R -> 20R
- R15: value 100R -> 330R
- R16, R17: value 240K -> 330R
- R18: value 1K5/DNP -> 330R
- R19, R20, R21: value 20K -> 330R
- R22: value 6K2 -> 10K
- R23: value 100K -> 240K
- R24: value 20K -> 240K
- R25: value 100K -> 10K
- R27, R28, R32: value 100R -> 20K
- R29: value 100R -> 6K2
- R30: value 100R -> 12K1
- R31, R33: value 100R -> 100K
- R34: value 10K -> 20K
- R35: value 10K -> 2K2/DNP
- R37: value 20R -> 2K2/DNP
- R39: value 20R -> 49R9
- R4, R81: value 2K2 -> 10K
- R40: value 20R -> 0R
- R41: value 0R -> 49R9
- R42: value 0R -> 2K2
- R44: value 100K -> 49R9
- R46: value 2K2 -> 49R9
- R47, R79: value 2K2 -> 20R
- R48: value 2K2/DNP -> 20R
- R49: value 2K2/DNP -> 0R/DNP
- R5: value 6K2 -> 2K2
- R50, R62: value 10K -> 100R
- R51: value 1K5/DNP -> 100R
- R52: value 470K -> 10K
- R53: value 0R -> 1K5/DNP
- R54, R55: value 0R -> 330R
- R56, R61: value 0R/DNP -> 100R
- R57, R60: value 0R -> 100R
- R58, R59: value 330R -> 100R
- R63: value 10K -> 100K
- R64: value 10K -> 6K2
- R65, R66: value 10K -> 0R
- R67, R69: value 330R -> 0R
- R68, R70: value 330R -> 0R/DNP
- R7: value 240K -> 10K
- R71, R72: value 330R -> 1K5/DNP
- R73: value 330R -> 240K
- R74: value 330R -> 10K
- R75: value 56K -> 10K
- R76: value 0R -> 10K
- R77, R80: value 2K2 -> 1K5/DNP
- R78: value 10K -> 20R
- R82: value 12K1 -> 10K
- R83: value 49R9 -> 10K
- U$11: value STM32F030F4P6 -> PIN-1X8; device alvie:TSSOP20 -> alvie:PIN-1X8
- U$12: value PIN-1X8 -> PIN-1X4; device alvie:PIN-1X8 -> alvie:PIN-1X4
- U$13: value PIN-1X8 -> PMS150C-U06; device alvie:PIN-1X8 -> alvie:SOT23-6
- U$14: value PN532_NFCB -> AP2000; device alvie:HW-147-NFC-NOHOLES -> alvie:SOT23-6
- U$15: value STM32F070F6 -> MT3608; device alvie:TSSOP20 -> alvie:SOT23-6
- U$16: value MIC550X -> PIN-1X10; device alvie:SOT23-5L -> alvie:PIN-1X10
- U$17: value PIN-1X4 -> PIN-1X10; device alvie:PIN-1X4 -> alvie:PIN-1X10
- U$25: value SR410361N -> PN532_NFCB; device alvie:LCD_7SEG_4DIGIT -> alvie:HW-147-NFC-NOHOLES
- U$26: value PIN-1X8 -> PIN-1X10; device alvie:PIN-1X8 -> alvie:PIN-1X10
- U$27: value TSSOP16 -> PIN-1X10; device alvie:TSSOP16 -> alvie:PIN-1X10
- U$28: value PFS154-S16 -> MIC550X; device alvie:SOIC16-N -> alvie:SOT23-5L
- U$29: value PIN-1X4 -> STM32F070F6; device alvie:PIN-1X4 -> alvie:TSSOP20
- U$3: value MT3608 -> SR410361N; device alvie:SOT23-6 -> alvie:LCD_7SEG_4DIGIT
- U$30: value CC2530 -> PIN-1X4; device alvie:RHA-S-PVQFN-N40 -> alvie:PIN-1X4
- U$6: value PIN-1X4 -> PIN-1X8; device alvie:PIN-1X4 -> alvie:PIN-1X8
- U$7: value PIN-1X8 -> PFS154-S16; device alvie:PIN-1X8 -> alvie:SOIC16-N
- U$8: value PMS150C-U06 -> PIN-1X4; device alvie:SOT23-6 -> alvie:PIN-1X4
- U$9: value PFS154-S16 -> TSSOP16; device alvie:SOIC16-N -> alvie:TSSOP16
- U1: value MIC550X -> STM32F107RCT6; device alvie:SOT23-5L -> ST Microelctronics_By_element14_Batch_1:QFP50P1200X1200X160-64N
- U2: value STM32F107RCT6 -> ESP-WROOM-32; device ST Microelctronics_By_element14_Batch_1:QFP50P1200X1200X160-64N -> esp32:ESP-WROOM-32
- U3: value ESP-WROOM-32 -> MIC550X; device esp32:ESP-WROOM-32 -> alvie:SOT23-5L
- moved H7 107.9 mm to (3.80, 3.80)
- moved C23 104.0 mm to (25.5, 88.5)
- moved C46 102.6 mm to (91.4, 26.8), flipped to the bottom, turned to 90 degrees
- moved C63 101.7 mm to (21.5, 10.8), turned to 0 degrees
- moved C48 101.4 mm to (98.3, 33.2), flipped to the bottom
- moved C35 101.1 mm to (11.5, 90.5), turned to 0 degrees
- moved C4 100.5 mm to (28.0, 80.0), flipped to the bottom
- moved C34 97.2 mm to (13.5, 85.0), turned to 0 degrees
- moved C1 97.0 mm to (34.5, 80.0), flipped to the bottom, turned to 180 degrees
- moved L11 96.7 mm to (94.5, 27.1), flipped to the bottom, turned to 180 degrees
- moved L1 95.7 mm to (34.4, 76.6), flipped to the bottom
- moved R43 93.5 mm to (6.50, 27.9), turned to 90 degrees
- moved H2 92.9 mm to (48.0, 96.0)
- moved C8 92.0 mm to (19.3, 95.0), flipped to the top, turned to 270 degrees
- moved C65 91.0 mm to (7.60, 70.5), turned to 180 degrees
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- renumbered T2 to T1
Connections:
- removed net +3V3_CC: C75.2, C76.2, C77.2, C78.2, C79.2, C80.2, C81.2, C83.2, L16.2, R87.1, U$30.10, U$30.21, U$30.24, U$30.27, U$30.28, U$30.29, U$30.31, U$30.39, U$31.4
- removed net CCLED1: R77.2, U$30.11
- removed net CCLED2: R81.2, U$30.9
- removed net CC_MISO: R76.2, U$30.37
- removed net CC_MOSI: R42.2, U$30.38
- removed net CC_SCK: R41.2, U$30.5
- removed net DEBUG_C: U$30.34, U$31.2
- removed net DEBUG_D: U$30.35, U$31.3
- removed net N$106: C85.2, Q12.1, U$30.32
- removed net N$79: C70.2, C73.2, L15.1
- removed net N$80: C71.1, U$30.25
- removed net N$82: C71.2, C72.2, L14.1
- removed net N$83: C73.1, C74.2, L14.2
- removed net N$84: C74.1, J7.S
- removed net N$85: R75.2, U$30.30
- removed net N$86: C82.2, U$30.40
- removed net N$87: LED8.C, R81.1
- removed net N$88: C86.2, Q13.3, U$30.23
- removed net N$89: C87.2, Q13.1, U$30.22
- removed net N$90: C84.2, Q12.3, U$30.33
- new net S0: U$16.1, X2.6
- new net S1: U$18.2, X2.7
- new net S10: U$18.5, X2.17
- new net S11: U$17.5, X2.18
- new net S12: U$16.5, X2.19
- new net S13: U$18.6, X2.20
- new net S14: U$17.6, X2.21
- new net S15: U$16.6, X2.22
- new net S16: U$18.7, X2.23
- new net S17: U$17.7, X2.24
- new net S18: U$16.7, X2.25
- new net S19: U$18.8, X2.26
- new net S2: U$17.2, X2.8
- new net S20: U$17.8, X2.27
- new net S21: U$16.8, X2.28
- new net S22: U$18.9, X2.30
- new net S23: U$17.9, X2.32
- new net S24: U$16.9, X2.34
- new net S25: U$18.10, X2.36
- new net S26: U$17.10, X2.38
- new net S27: U$16.10, X2.39
- new net S3: U$16.2, X2.9
- new net S4: U$18.3, X2.10
- new net S5: U$17.3, X2.12
- new net S6: U$16.3, X2.13
- new net S7: U$18.4, X2.14
- new net S8: U$17.4, X2.15
- new net S9: U$16.4, X2.16
- new net S_FB: R71.1, R72.2, U$14.3
- new net S_SW: L9.2, U$14.1
- new net S_VIN: C42.2, JP7.2, L9.1, U$14.4, U$14.6
- new net S_VOUT: C54.2, C55.2, JP8.1, R71.2, U$14.5
- new net VCC3: C71.2, C74.2, IC8.5, IC9.5, R77.2, U$26.10, U$26.9
- new net VCCI: C67.2, IC9.1, IC9.3, R77.1, U$27.10, U$27.9
- new net X0: IC8.1, U$26.2
- new net X1: IC8.2, U$26.3
- new net X10: IC8.13, U$27.5
- new net X11: IC8.11, U$27.6
- new net X12: IC8.10, U$27.7
- new net X13: IC8.9, U$27.8
- new net X2: IC8.3, U$26.4
- new net X3: IC8.4, U$26.5
- new net X4: IC8.6, U$26.6
- new net X5: IC8.7, U$26.7
- new net X6: IC8.8, U$26.8
- new net X7: IC8.16, U$27.2
- new net X8: IC8.15, U$27.3
- new net X9: IC8.14, U$27.4
- net +15V: now also C13.1, C57.1, C58.2, C59.2, D2.C, IC2.8, R73.2; no longer C11.1, C12.2, C13.2, C8.1, D3.C, IC1.8, R7.2
- net +3V3: now also C1.1, C10.2, C11.2, C15.2, C16.2, C17.2, C2.1, C22.1, C24.1, C27.1, C3.1, C30.2, C38.2, C39.2, C4.1, C47.1, C49.1, C52.1, C62.2, C64.2, C65.2, C76.2, C77.2, C79.2, C8.2, C80.2, IC1.1, IC1.19, IC1.9, IC4.4, J5.2, JP1.2, JP9.1, L1.1, L11.2, L12.1, L13.P$2, M3.3, Q1.2, Q2.2, Q5.2, Q7.2, R1.1, R10.2, R11.2, R22.2, R25.2, R35.2, R36.2, R37.2, R4.2, R52.2, R53.2, R54.2, R55.2, R63.1, R7.2, R75.2, R8.2, R83.2, U$10.4, U$19.16, U$22.2, U$23.7, U$25.VCC, U$25.VCC1, U$29.16, U$29.5, U$30.1, U$7.5, U$8.1, U1.1, U1.19, U1.32, U1.48, U1.64, U3.5, X1.2, X1.3; no longer C14.2, C15.1, C18.1, C19.1, C2.2, C26.1, C28.1, C30.1, C36.2, C4.2, C41.1, C42.1, C43.1, C45.1, C46.2, C51.2, C53.2, C54.2, C56.2, C59.2, C60.2, C61.2, C93.2, C94.2, C95.2, C96.2, IC11.1, IC11.19, IC11.9, IC15.4, J1.2, JP5.1, JP7.2, L10.1, L11.P$2, L16.1, L7.2, L8.1, LED7.A, LED8.A, M2.3, Q10.2, Q11.2, Q6.2, Q8.2, R18.2, R3.2, R34.2, R43.2, R44.1, R48.2, R49.2, R51.2, R52.1, R58.2, R59.2, R63.2, R64.2, R65.2, R66.2, R78.2, R79.2, R9.2, SV1.1, U$10.2, U$11.16, U$13.7, U$14.VCC, U$14.VCC1, U$15.16, U$15.5, U$16.5, U$17.1, U$29.4, U$33.1, U$6.1, U1.5, U2.1, U2.19, U2.32, U2.48, U2.64
- net +5V: now also C40.2, L7.1, USB2.P1; no longer C24.2, L4.1, USB1.P1
- net +5V_FILT: now also C43.1, L7.2, Q10.2, R64.2, U3.1, U3.3; no longer C25.1, L4.2, Q1.2, R5.2, U1.1, U1.3
- net A_MISO: now also J6.1; no longer J5.1
- net A_MOSI: now also J6.4; no longer J5.4
- net A_RESET: now also J6.5; no longer J5.5
- net A_SCK: now also J6.3; no longer J5.3
- net BOOT0: now also R43.2; no longer R10.2
- net CA0: now also Q1.1, R7.1, U$7.7; no longer Q8.1, R63.1, U$28.7
- net CA1: now also Q2.1, R11.1, U$7.6; no longer Q9.1, R64.1, U$28.6
- net CA2: now also Q3.1, R22.1, U$7.4; no longer Q10.1, R65.1, U$28.4
- net CA3: now also Q5.1, R25.1, U$7.3; no longer Q11.1, R66.1, U$28.3
- net CC_RST: now also U1.39, X1.22; no longer R87.2, U$30.20, U2.39
- net CC_RX: now also U1.53, X1.17; no longer U$30.17, U2.53
- net CC_SS: now also U1.40, X1.21; no longer U$30.6, U2.40
- net CC_TX: now also U1.54, X1.18; no longer U$30.16, U2.54
- net ESP_EN: now also U1.49, U2.3; no longer U2.49, U3.3
- net ESP_IO0: now also U1.29, U2.25; no longer U2.29, U3.25
- net ESP_MISO: now also R67.2, R68.2, U2.31; no longer R56.2, R57.2, R76.1, U3.31
- net ESP_MOSI: now also R69.2, R70.2, U2.37; no longer R42.1, R60.2, R61.2, U3.37
- net ESP_ON: now also Q9.1, R63.2; no longer Q6.1, R44.2
- net ESP_RX: now also U1.51, U2.34; no longer U2.51, U3.34
- net ESP_SCK: now also R66.2, U2.30; no longer R41.1, R55.2, U3.30
- net ESP_TX: now also U1.52, U2.35; no longer U2.52, U3.35
- net ESP_VCC: now also Q9.3, U2.2; no longer Q6.3, U3.2
- net GND: now also C1.2, C11.1, C15.1, C18.1, C19.1, C2.2, C21.1, C24.2, C28.1, C29.1, C3.2, C30.1, C31.1, C34.2, C35.2, C4.2, C40.1, C41.1, C42.1, C45.1, C47.2, C49.2, C5.1, C52.2, C53.2, C56.2, C58.1, C60.2, C62.1, C64.1, C66.2, C70.2, C71.1, C73.2, C74.1, C75.2, C8.1, D4.K, IC1.P, IC4.1, IC4.3, IC4.6, IC4.EXP, IC5.12, IC6.7, IC6.8, IC7.7, IC7.8, IC8.12, IC9.2, J1.2, J3.1, J4.2, J6.6, JP10.1, JP11.1, JP4.1, JP5.2, JP7.1, JP8.2, Q8.2, R23.1, R27.1, R29.1, R3.2, R30.1, R32.1, R34.1, R43.1, R72.1, R74.1, R76.1, S1.P$1, S2.P$2, U$12.3, U$12.4, U$13.2, U$14.2, U$15.2, U$18.1, U$19.15, U$20.12, U$22.1, U$23.8, U$25.GND, U$25.GND1, U$26.1, U$27.1, U$28.2, U$29.15, U$7.12, U$8.4, U1.12, U1.18, U1.31, U1.47, U1.63, U2.1, U2.15, U2.38, U2.GND, U3.2, X1.11, X1.29, X1.31, X1.33, X1.35, X1.37, X1.4, X1.40, X1.5, X2.11, X2.29, X2.31, X2.33, X2.35, X2.37, X2.4, X2.40, X2.5; no longer C1.1, C11.2, C13.1, C15.2, C18.2, C19.2, C2.1, C21.2, C24.1, C28.2, C29.2, C3.1, C30.2, C31.2, C34.1, C35.1, C4.1, C40.2, C41.2, C42.2, C45.2, C47.1, C49.1, C52.1, C53.1, C56.1, C58.2, C60.1, C62.2, C63.2, C64.2, C66.1, C75.1, C83.1, C84.1, C85.1, C86.1, C87.1, C93.1, C94.1, C95.1, C96.1, C97.1, C98.1, C99.1, D2.K, IC11.P, IC15.1, IC15.3, IC15.6, IC15.EXP, IC2.12, IC4.7, IC4.8, IC5.7, IC5.8, J3.2, J4.1, J5.6, J6.2, J7.GND@0, JP1.1, JP11.2, JP6.1, JP9.1, L15.2, Q12.2, Q12.4, Q13.2, Q13.4, Q4.2, R10.1, R16.1, R17.1, R20.1, R22.1, R26.1, R35.1, R38.1, R50.2, R75.1, R8.1, S1.P$2, S2.P$1, SV1.3, SV1.4, U$11.15, U$13.8, U$14.GND, U$14.GND1, U$15.15, U$16.2, U$17.4, U$28.12, U$29.1, U$3.2, U$30.1, U$30.2, U$30.3, U$30.EXP, U$31.1, U$32.1, U$6.4, U$8.2, U$9.12, U1.2, U2.12, U2.18, U2.31, U2.47, U2.63, U3.1, U3.15, U3.38, U3.GND
- net LCLK: now also U$10.2, U$7.11; no longer U$28.11, U$29.2
- net LDAT: now also U$10.3, U$7.13; no longer U$28.13, U$29.3
- net LED0: now also R2.2; no longer R1.2
- net LED1: now also R5.2; no longer R2.2
- net LED2: now also R9.2; no longer R4.2
- net MCO: now also R40.1, U1.41; no longer R53.1, U2.41
- net MCU_MISO: now also IC5.7, R59.1, R60.1, U$13.3, U$20.7; no longer IC2.7, R30.1, R31.1, U$8.3, U$9.7
- net MCU_MOSI: now also IC5.10, R61.1, R62.1, U$13.1, U$20.10; no longer IC2.10, R32.1, R33.1, U$8.1, U$9.10
- net MCU_PA0: now also IC5.11, R56.1, U$20.11; no longer IC2.11, R27.1, U$9.11
- net MCU_PA7: now also IC5.6, R57.1, U$20.6; no longer IC2.6, R28.1, U$9.6
- net MCU_SCK: now also IC5.9, R58.1, U$13.6, U$20.9; no longer IC2.9, R29.1, U$8.6, U$9.9
- net MISO: now also R59.2, R62.2; no longer R30.2, R33.2
- net MOSI: now also R60.2, R61.2; no longer R31.2, R32.2
- net N$1: now also R5.1; no longer R2.1
- net N$10: now also C45.2, C46.2, L11.1, U$19.5; no longer C34.2, C35.2, L7.1, U$11.5
- net N$100: now also IC3.13, U$11.5, U$9.12; no longer IC6.13, U$26.5, U$27.12
- net N$101: now also IC3.14, U$11.6, U$9.11; no longer IC6.14, U$26.6, U$27.11
- net N$102: now also IC3.12, U$11.4, U$9.13; no longer IC6.12, U$26.4, U$27.13
- net N$103: now also IC3.11, U$11.3, U$9.14; no longer IC6.11, U$26.3, U$27.14
- net N$104: now also IC3.10, U$11.2, U$9.15; no longer IC6.10, U$26.2, U$27.15
- net N$105: now also IC3.9, U$11.1, U$9.16; no longer IC6.9, U$26.1, U$27.16
- net N$11: now also C36.2, JP6.1, L6.2; no longer C20.2, JP4.1, L3.2
- net N$13: now also C41.2, J4.1, J5.1, L8.1; no longer C32.2, J2.1, J3.1, L6.1
- net N$14: now also C37.2, JP6.2; no longer C23.2, JP4.2
- net N$15: now also L6.1, Q7.3, Q8.3; no longer L3.1, Q3.3, Q4.3
- net N$16: now also L8.2, M3.2; no longer L6.2, M2.2
- net N$17: now also L14.1; no longer L12.1
- net N$18: now also Q7.1, R49.1, R50.1; no longer Q3.1, R13.1, R14.1
- net N$19: now also Q8.1, R51.1; no longer Q4.1, R15.1
- net N$2: now also C44.2, L10.P$1, Q10.3, U$15.4, U$15.5; no longer C6.2, L2.P$1, Q1.3, U$3.4, U$3.5
- net N$20: now also R12.1, USB1.P2; no longer R39.1, USB2.P2
- net N$21: now also R2.1; no longer R1.1
- net N$22: now also R14.1, USB1.P3; no longer R40.1, USB2.P3
- net N$23: now also JP9.2, R76.2, U$19.1; no longer JP5.2, R35.2, U$11.1
- net N$24: now also U$12.1, X2.1; no longer LED7.C, R77.1
- net N$25: now also R65.2, U2.29; no longer R54.2, U3.29
- net N$26: now also R38.1; no longer R45.1
- net N$27: now also R42.1; no longer R46.1
- net N$28: now also R45.1; no longer R47.1
- net N$29: now also R78.1; no longer R36.1
- net N$3: now also R9.1; no longer R4.1
- net N$30: now also IC5.16; no longer IC2.16
- net N$31: now also IC5.15; no longer IC2.15
- net N$32: now also IC5.14; no longer IC2.14
- net N$33: now also R79.1; no longer R37.1
- net N$34: now also IC6.3, IC7.3; no longer IC4.3, IC5.3
- net N$35: now also IC5.13; no longer IC2.13
- net N$36: now also R47.1, USB2.P2; no longer R11.1, USB1.P2
- net N$37: now also R48.1, USB2.P3; no longer R12.1, USB1.P3
- net N$38: now also IC6.4, JP12.1; no longer IC4.4, JP8.1
- net N$39: now also L4.1, USB1.P1; no longer L9.1, USB2.P1
- net N$4: now also L2.2; no longer L1.2
- net N$40: now also IC1.24, R30.2; no longer IC11.24, R82.2
- net N$41: now also C6.2, J1.1, L3.1; no longer C66.2, J6.1, L13.1
- net N$42: now also R73.1, R74.2, U$15.3; no longer R7.1, R8.2, U$3.3
- net N$43: now also C63.2, D3.K, D4.A; no longer C5.2, D1.K, D2.A
- net N$44: now also C35.1; no longer C57.1
- net N$45: now also C34.1; no longer C58.1
- net N$46: now also R54.1; no longer R58.1
- net N$47: now also L3.2, M2.2; no longer L13.2, M3.2
- net N$48: now also C18.2, JP5.1, M2.3; no longer C67.2, JP11.1, M3.3
- net N$49: now also IC7.13, JP13.8; no longer IC5.13, JP10.8
- net N$5: now also C5.2, J2.1, JP3.2, L2.1; no longer C1.2, J1.1, JP2.2, L1.1
- net N$50: now also IC2.6, R28.2, R29.2; no longer IC1.6, R21.2, R22.2
- net N$51: now also IC2.2, R26.2, R27.2; no longer IC1.2, R19.2, R20.2
- net N$52: now also IC6.13, JP12.8; no longer IC4.13, JP8.8
- net N$53: now also R55.1; no longer R59.1
- net N$54: now also IC5.1; no longer IC2.1
- net N$55: now also IC5.2; no longer IC2.2
- net N$56: now also C28.2, L5.2, R39.2, R41.2, R44.2, R46.2; no longer C99.2, L10.2, R83.2, R84.2, R85.2, R86.2
- net N$57: now also IC5.3; no longer IC2.3
- net N$58: now also C21.2, C23.2, IC1.6; no longer C97.2, C98.2, IC11.6
- net N$59: now also IC5.4; no longer IC2.4
- net N$60: now also IC6.14, JP12.7; no longer IC4.14, JP8.7
- net N$61: now also IC6.12, JP12.5; no longer IC4.12, JP8.5
- net N$62: now also IC6.1, JP12.4; no longer IC4.1, JP8.4
- net N$63: now also IC6.5, JP12.3; no longer IC4.5, JP8.3
- net N$64: now also IC6.2, JP12.2; no longer IC4.2, JP8.2
- net N$65: now also Q2.3, U$3.9; no longer Q9.3, U$25.9
- net N$66: now also J6.2; no longer J5.2
- net N$67: now also IC7.14, JP13.7; no longer IC5.14, JP10.7
- net N$68: now also IC7.15, JP13.6; no longer IC5.15, JP10.6
- net N$69: now also IC7.12, JP13.5; no longer IC5.12, JP10.5
- net N$7: now also C14.2; no longer C3.2
- net N$70: now also IC6.15, JP12.6; no longer IC4.15, JP8.6
- net N$71: now also IC7.1, JP13.4; no longer IC5.1, JP10.4
- net N$72: now also IC7.5, JP13.3; no longer IC5.5, JP10.3
- net N$73: now also IC7.2, JP13.2; no longer IC5.2, JP10.2
- net N$74: now also IC7.4, JP13.1; no longer IC5.4, JP10.1
- net N$75: now also Q3.3, U$3.8; no longer Q10.3, U$25.8
- net N$76: now also Q1.3, U$3.12; no longer Q8.3, U$25.12
- net N$77: now also Q5.3, U$3.6; no longer Q11.3, U$25.6
- net N$78: now also U$12.2, U$17.1, X2.2, X2.3; no longer C70.1, U$30.26
- net N$8: now also C29.2, R36.1, U$8.2; no longer C10.2, R9.1, U$6.2
- net N$81: now also IC3.8, U$6.1, U$9.1; no longer IC6.8, U$27.1, U$7.1
- net N$91: now also IC3.7, U$6.2, U$9.2; no longer IC6.7, U$27.2, U$7.2
- net N$92: now also IC3.6, U$6.3, U$9.3; no longer IC6.6, U$27.3, U$7.3
- net N$93: now also IC3.5, U$6.4, U$9.4; no longer IC6.5, U$27.4, U$7.4
- net N$94: now also IC3.4, U$6.5, U$9.5; no longer IC6.4, U$27.5, U$7.5
- net N$95: now also IC3.3, U$6.6, U$9.6; no longer IC6.3, U$27.6, U$7.6
- net N$96: now also IC3.2, U$6.7, U$9.7; no longer IC6.2, U$27.7, U$7.7
- net N$97: now also IC3.1, U$6.8, U$9.8; no longer IC6.1, U$27.8, U$7.8
- net N$98: now also IC3.16, U$11.8, U$9.9; no longer IC6.16, U$26.8, U$27.9
- net N$99: now also IC3.15, U$11.7, U$9.10; no longer IC6.15, U$26.7, U$27.10
- net NBOOT0: now also R82.2, U$29.1; no longer R38.2, U$15.1
- net NIRQ: now also U$25.IRQ, U$29.7; no longer U$14.IRQ, U$15.7
- net NLED0: now also R38.2, U1.46; no longer R45.2, U2.46
- net NLED1: now also R42.2, U1.35; no longer R46.2, U2.35
- net NLED2: now also R45.2, U1.36; no longer R47.2, U2.36
- net NNRST: now also R83.1, U$29.4; no longer R43.1, U$15.4
- net NOSC_IN: now also C81.2, Q11.2, U$29.2; no longer C47.2, Q7.2, U$15.2
- net NOSC_OUT: now also C82.2, Q11.1, U$29.3; no longer C52.2, Q7.1, U$15.3
- net NRST: now also R52.1, S2.P$1; no longer R6.1, S1.P$1
- net NRSTO: now also U$25.RSTO, U$29.6; no longer U$14.RSTO, U$15.6
- net NSWCLK: now also U$29.20, U$30.3; no longer U$15.20, U$17.3
- net NSWDIO: now also U$29.19, U$30.2; no longer U$15.19, U$17.2
- net NUSBDM: now also R78.2, U$29.17; no longer R36.2, U$15.17
- net NUSBDP: now also R79.2, R80.1, U$29.18; no longer R37.2, R51.1, U$15.18
- net N_MISO: now also U$25.MISO, U$29.12; no longer U$14.MISO, U$15.12
- net N_MOSI: now also U$25.MOSI, U$29.13; no longer U$14.MOSI, U$15.13
- net N_RX: now also U$25.SDA/TX, U$29.9; no longer U$14.SDA/TX, U$15.9
- net N_SCK: now also U$25.SCK, U$29.11; no longer U$14.SCK, U$15.11
- net N_SS: now also U$25.SS, U$29.10; no longer U$14.SS, U$15.10
- net N_TX: now also U$25.SCL/RX, U$29.8; no longer U$14.SCL/RX, U$15.8
- net OSC_IN: now also C31.2, Q6.2; no longer C16.2, Q2.2
- net OSC_OUT: now also C32.2, Q6.1; no longer C17.2, Q2.1
- net PA0: now also U$19.6, U$23.3; no longer U$11.6, U$13.3
- net PA1: now also U$19.7, U$23.2; no longer U$11.7, U$13.2
- net PA10: now also U$19.18; no longer U$11.18
- net PA13: now also U$19.19, U$21.2; no longer U$11.19, U$12.2
- net PA14: now also U$19.20, U$21.1; no longer U$11.20, U$12.1
- net PA15/NSS: now also R65.1, U1.50; no longer R54.1, U2.50
- net PA2: now also U$19.8, U$23.1; no longer U$11.8, U$13.1
- net PA3: now also U$19.9, U$21.8; no longer U$11.9, U$12.8
- net PA3/ADC3: now also U1.17, X1.30; no longer U$33.2, U2.17
- net PA4: now also U$19.10, U$21.7; no longer U$11.10, U$12.7
- net PA4/DAC1: now also U1.20, X1.32; no longer U$33.3, U2.20
- net PA5: now also U$19.11, U$21.6; no longer U$11.11, U$12.6
- net PA5/DAC2: now also U1.21, X1.34; no longer U$32.3, U2.21
- net PA6: now also U$19.12, U$21.5; no longer U$11.12, U$12.5
- net PA7: now also U$19.13, U$21.4; no longer U$11.13, U$12.4
- net PA9: now also U$19.17; no longer U$11.17
- net PB1: now also U$19.14, U$21.3; no longer U$11.14, U$12.3
- net PB6/UART1_TX: now also U1.58, X1.12; no longer SV1.24, U2.58
- net PB7/UART1_RX: now also U1.59, X1.13; no longer SV1.23, U2.59
- net PEDAL: now also JP11.2, R81.1; no longer JP9.2, R62.1
- net PF0: now also U$19.2, U$23.6; no longer U$11.2, U$13.6
- net PF1: now also U$19.3, U$23.5; no longer U$11.3, U$13.5
- net PHY_LED0: now also IC1.3; no longer IC11.3
- net PHY_LED1: now also IC1.2; no longer IC11.2
- net PWM1: now also R50.2, R51.2; no longer R14.2, R15.2
- net PWM2: now also R49.2; no longer R13.2
- net PWRON: now also Q10.1, R64.1; no longer Q1.1, R5.1
- net REG33IN: now also C51.2, D1.1, IC4.5, IC4.7, IC4.8, J3.3, X1.1; no longer C49.2, D4.1, IC15.5, IC15.7, IC15.8, J4.3, SV1.2
- net RMII_CRS_DV: now also IC1.11, U1.23; no longer IC11.11, U2.23
- net RMII_MDC: now also IC1.13, R8.1, U1.9; no longer IC11.13, R79.1, U2.9
- net RMII_MDIO: now also IC1.12, R10.1, U1.16; no longer IC11.12, R80.1, U2.16
- net RMII_NRST: now also IC1.15, R4.1, U1.22; no longer IC11.15, R78.1, U2.22
- net RMII_REF_CLK: now also IC1.14, U1.15; no longer IC11.14, U2.15
- net RMII_RXD0: now also IC1.8, U1.24; no longer IC11.8, U2.24
- net RMII_RXD1: now also IC1.7, U1.25; no longer IC11.7, U2.25
- net RMII_TXD0: now also IC1.17, U1.33; no longer IC11.17, U2.33
- net RMII_TXD1: now also IC1.18, U1.34; no longer IC11.18, U2.34
- net RMII_TX_EN: now also IC1.16, U1.30; no longer IC11.16, U2.30
- net RX: now also JP4.2; no longer JP3.2
- net RXM1: now also IC1.20, R41.1; no longer IC11.20, R84.1
- net RXP1: now also IC1.21, R39.1; no longer IC11.21, R83.1
- net SA: now also R13.2, U$3.11; no longer R67.2, U$25.11
- net SB: now also R15.2, U$3.7; no longer R68.2, U$25.7
- net SC: now also R16.2, U$3.4; no longer R69.2, U$25.4
- net SCK: now also R58.2; no longer R29.2
- net SD: now also R17.2, U$3.2; no longer R70.2, U$25.2
- net SDP: now also R21.2, U$3.3; no longer R74.2, U$25.3
- net SE: now also R18.2, U$3.1; no longer R71.2, U$25.1
- net SEG_A: now also R13.1, U$7.9; no longer R67.1, U$28.9
- net SEG_B: now also R15.1, U$7.14; no longer R68.1, U$28.14
- net SEG_C: now also R16.1, U$7.2; no longer R69.1, U$28.2
- net SEG_D: now also R17.1, U$7.15; no longer R70.1, U$28.15
- net SEG_DP: now also R21.1, U$7.16; no longer R74.1, U$28.16
- net SEG_E: now also R18.1, U$7.10; no longer R71.1, U$28.10
- net SEG_F: now also R19.1, U$7.8; no longer R72.1, U$28.8
- net SEG_G: now also R20.1, U$7.1; no longer R73.1, U$28.1
- net SEL_A0: now also IC7.11; no longer IC5.11
- net SEL_A1: now also IC6.11; no longer IC4.11
- net SEL_B0: now also IC7.10; no longer IC5.10
- net SEL_B1: now also IC6.10; no longer IC4.10
- net SEL_C0: now also IC7.9; no longer IC5.9
- net SEL_C1: now also IC6.9; no longer IC4.9
- net SEL_INH: now also IC6.6, IC7.6; no longer IC4.6, IC5.6
- net SF: now also R19.2, U$3.10; no longer R72.2, U$25.10
- net SG: now also R20.2, U$3.5; no longer R73.2, U$25.5
- net STM_PA0: now also R56.2; no longer R27.2
- net STM_PA7: now also R57.2; no longer R28.2
- net SW: now also JP2.2, R6.1; no longer JP1.2, R3.1
- net SWIM: now also U$8.3; no longer U$6.3
- net TX: now also JP4.3; no longer JP3.3
- net TXM1: now also IC1.22, R46.1; no longer IC11.22, R86.1
- net TXP1: now also IC1.23, R44.1; no longer IC11.23, R85.1
- net UART1RX: now also U1.43, X1.19; no longer SV1.18, U2.43
- net UART1TX: now also U1.42, X1.20; no longer SV1.17, U2.42
- net USBDM: now also R47.2; no longer R11.2
- net USBDP: now also R48.2, R53.1; no longer R12.2, R18.1
- net USBPWR: now also D1.2, L4.2; no longer D4.2, L9.2
- net USBPWR1: now also C78.2, L14.2, U$28.1, U$28.3; no longer C55.2, L12.2, U$16.1, U$16.3
- net VDDA: now also C56.1, L12.2; no longer C31.1, L5.2
- net VDD_OUT: now also C25.1, C53.1, IC2.1, IC5.5, R26.1, R33.2, U$13.5, U$20.5; no longer C21.1, C27.1, IC1.1, IC2.5, R19.1, R25.2, U$8.5, U$9.5
- net VDD_PWM: now also IC2.3, R23.2; no longer IC1.3, R16.2
- net VDD_SENS: now also R33.1, R34.2; no longer R25.1, R26.2
- net VEE: now also C13.2, C66.1, D3.A, IC2.4; no longer C7.1, C8.2, D1.A, IC1.4
- net VNEG_PWM: now also C63.1; no longer C5.1
- net VPP_OUT: now also C26.1, C60.1, IC2.7, IC5.8, R28.1, R31.2, U$13.4, U$20.8; no longer C22.1, C29.1, IC1.7, IC2.8, R21.1, R23.2, U$8.4, U$9.8
- net VPP_PWM: now also IC2.5, R24.2; no longer IC1.5, R17.2
- net VPP_SENS: now also R31.1, R32.2; no longer R23.1, R24.2
- net VSW: now also D2.A, L10.P$2, U$15.1; no longer D3.A, L2.P$2, U$3.1
- net V_BATT: now also C70.1, C72.2, C73.1, C75.1, IC6.16, IC7.16, JP10.2, R81.2; no longer C62.1, C63.1, C64.1, C65.2, IC4.16, IC5.16, JP6.2, R62.2
- net XBOOT0: now also JP1.1, R3.1, U1.60; no longer JP7.1, R50.1, U2.60
- net XI: now also IC1.5, R40.2; no longer IC11.5, R53.2
- net XNRST: now also C61.2, R75.1, U$19.4, U$23.4; no longer C37.2, R34.1, U$11.4, U$13.4
- net XOSC_IN: now also C19.2, Q4.2, U1.5; no longer C38.2, Q5.2, U2.5
- net XOSC_OUT: now also C20.2, Q4.1, U1.6; no longer C39.2, Q5.1, U2.6
- net XPA0: now also U1.14, X1.28; no longer SV1.12, U2.14
- net XPB0/ADC8: now also U1.26, X1.36; no longer U$32.2, U2.26
- net XPB1: now also U1.27, X1.38; no longer U$33.4, U2.27
- net XPB2: now also U1.28, X1.39; no longer U$32.4, U2.28
- net XPC0: now also U1.8, X1.25; no longer SV1.13, U2.8
- net XPC13: now also U1.2, X1.14; no longer SV1.22, U2.2
- net XPC14: now also U1.3, X1.15; no longer SV1.19, U2.3
- net XPC15: now also U1.4, X1.16; no longer SV1.20, U2.4
- net XPC2: now also U1.10, X1.26; no longer SV1.14, U2.10
- net XPC3: now also U1.11, X1.27; no longer SV1.11, U2.11
- net XPC6: now also U1.37, X1.24; no longer SV1.15, U2.37
- net XPC7: now also U1.38, X1.23; no longer SV1.16, U2.38
- net XSCL: now also R35.1, U$22.3, U1.61, X1.6; no longer R48.1, SV1.26, U$10.3, U2.61
- net XSDA: now also R37.1, U$22.4, U1.62, X1.7; no longer R49.1, SV1.25, U$10.4, U2.62
- net XSPI_MISO: now also R67.1, R70.1, U1.56, X1.9; no longer R57.1, R61.1, U2.56
- net XSPI_MOSI: now also R68.1, R69.1, U1.57, X1.10; no longer R56.1, R60.1, U2.57
- net XSPI_SCK: now also R66.1, U1.55, X1.8; no longer R55.1, U2.55
- net XSW: now also IC4.2, L13.P$1; no longer IC15.2, L11.P$1
- net XUSBDM: now also R12.2, U1.44; no longer R39.2, U2.44
- net XUSBDP: now also R14.2, U1.45; no longer R40.2, U2.45
- net XVDDA: now also C12.2, C7.1, L1.2, U1.13; no longer C40.1, C44.2, L8.2, U2.13
- net XXNRST: now also R1.2, S1.P$2, U1.7; no longer R52.2, S2.P$2, U2.7
Routing:
- net GND: track 139.0 -> 193.1 mm, vias 351 -> 342
- net +3V3_CC: track 52.2 -> 0.00 mm, vias 8 -> 0
- net +3V3: track 695.3 -> 729.9 mm, vias 40 -> 44
- net XSPI_MISO: track 10.4 -> 41.8 mm, vias 1 -> 2
- net XSPI_MOSI: track 13.5 -> 42.5 mm
- net XSPI_SCK: track 8.16 -> 36.5 mm
- net DEBUG_C: track 24.2 -> 0.00 mm
- net VCC3: track 0.00 -> 20.4 mm
- net N$90: track 17.0 -> 0.00 mm
- net XPC13: track 30.2 -> 13.5 mm
- net N$24: track 0.00 -> 15.5 mm
- net VCCI: track 0.00 -> 14.8 mm
- net DEBUG_D: track 14.6 -> 0.00 mm
- net XPB1: track 9.18 -> 23.5 mm, vias 2 -> 4
- net N$78: track 3.90 -> 18.0 mm, vias 0 -> 1
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- added copper zone on layer 1, net S_SW
- added copper zone on layer 1, net S_VIN
Other:
- board text added: "3V3"
- board text added: "STEPUP"
- board text added: "VIN"
- board text added: "VO"
- board text added: "Vout=1.23 x ( 1 + R41/R42 )"

Commit message: Production
Parts:
- C39, C67: value (none) -> 22uF
- C42, C55, C72: value (none) -> 10uF
- C70, C73, C75: value (none) -> 100nF
- L1: value 10mH -> 10uH
- L6: value (none) -> 150nH
- moved H3 0.50 mm to (48.0, 54.0)
- moved C18 0.40 mm to (74.0, 25.6)
Routing:
- net GND: vias 342 -> 343
Other:
- board text added: "ALD192/1-1"
- board text added: "ALD192/2-1"
- board text added: "ALD192/4-1"
- board text added: "ALD192/5-1"
- board text added: "ALD192/6-1"
- board text added: "ALD192/7-1"
- board text added: "ALD192/8-1"
- board text added: "ALD192/9-1"
- board text added: "ALD193/3-1"
