File: misc_designs/padaukprog.sch (EAGLE design)
At the start: 320 parts, among them IC1 LM358D, IC11 LAN8720A, IC15 TPS62063, IC4 4051D, IC5 4051D, IC6 IC_DIL16-SOIC-16, J1 JUMPER_SOLDER_1X2, J2 JUMPER_SOLDER_1X2, J3 JST-PH 2mm, J5 AVR_SPI_PRG_6NS, J6 JST-PH 2mm, J7 CON-HIROSE-COAXIAL-U.FL, M1 XT1861B, M2 XT1861B, M3 XT1861B, P1 B3B-PH-K, P2 B3B-PH-K, Q1 BSS84, Q10 BSS84, Q11 BSS84, Q12 CRISTAL-3225, Q13 CRISTAL-3225, Q2 8MHz, Q3 BSS84, Q4 BSS123, Q5 25MHz, Q6 FDN338, Q7 8MHz, Q8 BSS84, Q9 BSS84, T2 Hanrun HR917550A, U1 MIC550X, U2 STM32F107RCT6, U3 ESP-WROOM-32, U4 ATTINY24A-SSU

Commit message: Final routed
Parts:
- removed C83: (no value), GadgetFactory:C0805
- removed C84, C85, C86, C87: 15pF, GadgetFactory:C0402
- removed C93, C94, C95: 100nF, GadgetFactory:C0603
- removed C96: 2.2uF, GadgetFactory:C0805
- removed C97: 1uF, GadgetFactory:C0603
- removed C98: 1nF, GadgetFactory:C0603
- removed C99: 100nF/DNP, GadgetFactory:C0603
- removed H8: MOUNT-PAD-ROUND3.2, holes:MOUNT-PAD-ROUND3.2
- removed IC11: LAN8720A, sigedi-footprints:LAN8720A
- removed IC15: TPS62063, alvie:TPS62063
- removed J7: CON-HIROSE-COAXIAL-U.FL, m-pad-2.1:CON-HIROSE-COAXIAL-U.FL
- removed L15: (no value), GadgetFactory:L0402
- removed L16: 600R, GadgetFactory:L0805
- removed LED7, LED8: LG L29K-G2J1-24, dp_devices:LED-0603
- removed Q12, Q13: CRISTAL-3225, alvie:CRISTAL-3225
- removed R84, R85, R86: 49R9, GadgetFactory:R0603
- removed R87: 10K, GadgetFactory:R0603
- removed SV1: MA13-2W, alvie:MA13-2W
- removed U$31, U$32, U$33: PIN-1X4, alvie:PIN-1X4
- added H6: MOUNT-PAD-ROUND3.2, holes:MOUNT-PAD-ROUND3.2
- added IC3: IC_DIL16-SOIC-16, dp_devices:IC_DIL16-SOIC-16
- added IC7: 4051D, 40xx:4051D
- added IC8, U$20: PFS154-S16, alvie:PFS154-S16
- added IC9: MIC550X, alvie:MIC550X
- added JP12, JP13, U$21, U$23: PIN-1X8, alvie:PIN-1X8
- added U$18: PIN-1X10, alvie:PIN-1X10
- added U$19: STM32F030F4P6, alvie:STM32F030F4P6
- added U$22: PIN-1X4, alvie:PIN-1X4
- added X1, X2: FH12-40S-0.5SH, con-hirose:FH12-40S-0.5SH
- C1: value 22uF 16V -> 100nF 6.3V; device GadgetFactory:C0805 -> GadgetFactory:C0603
- C11, C29, C8: value 100nF 50V -> 100nF
- C12: value 22uF 50V -> 10uF; device GadgetFactory:C0805 -> GadgetFactory:C0603
- C13: value 22uF 50V -> 2.2uF 50V
- C14: value 100nF -> 2.2uF
- C15, C45: value 100nF 6.3V -> 100nF
- C16: value 20pF 6.3V -> 2.2uF; device GadgetFactory:C0603 -> GadgetFactory:C0805
- C17: value 20pF 6.3V -> 10uF
- C18: value 100nF 6.3V -> 10uF
- C19: value 100nF 6.3V -> 16pF 6.3V
- C2: value 100nF -> 100nF 6.3V
- C20: value 1uF -> 16pF 6.3V
- C21: value 100nF 50V -> 1uF
- C22, C27, C7: value 100nF 50V -> 100nF 6.3V
- C23: value 10uF -> 1nF; device GadgetFactory:C0805 -> GadgetFactory:C0603
- C24: value 22uF -> 100nF 6.3V; device GadgetFactory:C0805 -> GadgetFactory:C0603
- C25: value 10uF 6.3V -> 100nF 50V
- C26: value 100nF 6.3V -> 100nF 50V
- C28: value 10uF 6.3V -> 100nF/DNP
- C3: value 2.2uF -> 100nF 6.3V
- C30: value 10uF 6.3V -> 100nF
- C31: value 100nF 6.3V -> 20pF 6.3V
- C32: value 22uF 16V -> 20pF 6.3V; device GadgetFactory:C0805 -> GadgetFactory:C0603
- C33: value 10uF -> 100nF
- C34, C76: value 1uF -> 100nF
- C36, C61: value 100nF -> 1uF
- C37: value 1uF -> 10uF; device GadgetFactory:C0603 -> GadgetFactory:C0805
- C38: value 16pF 6.3V -> 10uF
- C39: value 16pF 6.3V -> (none); device GadgetFactory:C0603 -> GadgetFactory:C0805
- C4: value 10uF -> 100nF 6.3V
- C40: value 100nF 6.3V -> 22uF; device GadgetFactory:C0603 -> GadgetFactory:C0805
- C41: value 100nF 6.3V -> 22uF 16V; device GadgetFactory:C0603 -> GadgetFactory:C0805
- C42: value 100nF 6.3V -> (none); device GadgetFactory:C0603 -> GadgetFactory:C0805
- C43: value 100nF 6.3V -> 10uF 6.3V
- C44: value 10uF -> 22uF 16V; device GadgetFactory:C0603 -> GadgetFactory:C0805
- C46: value 10uF -> 1uF
- C47: value 20pF 6.3V -> 100nF 6.3V
- C48: value 10uF -> 10uF; device GadgetFactory:C0805 -> GadgetFactory:C0603
- C49: value 10uF -> 10uF 6.3V; device GadgetFactory:C0805 -> GadgetFactory:C0603
- C5: value 100nF 50V -> 22uF 16V; device GadgetFactory:C0603 -> GadgetFactory:C0805
- C51: value 10nF -> 10uF; device GadgetFactory:C0603 -> GadgetFactory:C0805
- C52: value 20pF 6.3V -> 10uF 6.3V
- C53, C57, C60: value 100nF -> 100nF 50V
- C55: value 10uF -> (none)
- C56: value 10nF -> 100nF 6.3V
- C58, C59: value 100nF -> 22uF 50V; device GadgetFactory:C0603 -> GadgetFactory:C0805
- C62: value (none) -> 10uF; device GadgetFactory:C0603 -> GadgetFactory:C0805
- C63: value (none) -> 100nF 50V
- C64: value (none) -> 100nF
- C65: value (none) -> 10nF; device GadgetFactory:C0805 -> GadgetFactory:C0603
- C66: value 22uF 16V -> 100nF 50V; device GadgetFactory:C0805 -> GadgetFactory:C0603
- C67: value 10uF -> (none); device GadgetFactory:C0603 -> GadgetFactory:C0805
- C69: value (none) -> 100nF; device GadgetFactory:C0805 -> GadgetFactory:C0603
- C70, C73, C77, C80: device GadgetFactory:C0402 -> GadgetFactory:C0603
- C71, C74: value (none) -> 100nF; device GadgetFactory:C0402 -> GadgetFactory:C0603
- C72: device GadgetFactory:C0402 -> GadgetFactory:C0805
- C75: value 100nF -> (none)
- C78: value 100nF -> 10uF; device GadgetFactory:C0402 -> GadgetFactory:C0805
- C79: value 220pF -> 10nF; device GadgetFactory:C0402 -> GadgetFactory:C0603
- C81: value 100nF -> 20pF 6.3V; device GadgetFactory:C0402 -> GadgetFactory:C0603
- C82: value 1uF -> 20pF 6.3V
- C9: value 2.2uF 50V -> 100nF 50V; device GadgetFactory:C0805 -> GadgetFactory:C0603
- D1: value RB521S-30 -> 1N4148W; device GadgetFactory:DIODE-SCHOTTKY_SOD523 -> alvie:1N4148W
- D2: value RB521S-30 -> 2SS100L-W; device GadgetFactory:DIODE-SCHOTTKY_SOD523 -> dp_devices:DIODE-SOD-123
- D3: value 2SS100L-W -> RB521S-30; device dp_devices:DIODE-SOD-123 -> GadgetFactory:DIODE-SCHOTTKY_SOD523
- D4: value 1N4148W -> RB521S-30; device alvie:1N4148W -> GadgetFactory:DIODE-SCHOTTKY_SOD523
- IC1: value LM358D -> LAN8720A; device linear:LM358D -> sigedi-footprints:LAN8720A
- IC2: value (none) -> LM358D; device ic-package:DIL16 -> linear:LM358D
- IC4: value 4051D -> TPS62063; device 40xx:4051D -> alvie:TPS62063
- IC5: value 4051D -> (none); device 40xx:4051D -> ic-package:DIL16
- IC6: value IC_DIL16-SOIC-16 -> 4051D; device dp_devices:IC_DIL16-SOIC-16 -> 40xx:4051D
- J1: value JUMPER_SOLDER_1X2 -> JST-PH 2mm; device dp_devices:JUMPER_SOLDER_1X2 -> SparkFun-Connectors:CONN_02JST-PTH-2
- J3: value JST-PH 2mm -> (none); device SparkFun-Connectors:CONN_02JST-PTH-2 -> GadgetFactory:JACK-PLUG
- J4: value (none) -> JST-PH 2mm; device GadgetFactory:JACK-PLUG -> SparkFun-Connectors:CONN_02JST-PTH-2
- J5: value AVR_SPI_PRG_6NS -> JUMPER_SOLDER_1X2; device SparkFun-Connectors:AVR_SPI_PRG_6NS -> dp_devices:JUMPER_SOLDER_1X2
- J6: value JST-PH 2mm -> AVR_SPI_PRG_6NS; device SparkFun-Connectors:CONN_02JST-PTH-2 -> SparkFun-Connectors:AVR_SPI_PRG_6NS
- JP10: value PIN-1X8 -> VBat +; device alvie:PIN-1X8 -> alvie:PIN-1X2
- JP11: value PIN-1X2 -> Pedal
- JP3: value PIN-1X3 -> PIN-1X2; device alvie:PIN-1X3 -> alvie:PIN-1X2
- JP4: value PIN-1X2 -> PIN-1X3; device alvie:PIN-1X2 -> alvie:PIN-1X3
- JP6: value VBat + -> PIN-1X2
- JP8: value PIN-1X8 -> PIN-1X2; device alvie:PIN-1X8 -> alvie:PIN-1X2
- JP9: value Pedal -> PIN-1X2
- L1: value 10uH -> 10mH
- L10: value 600R -> DFE252012F; device GadgetFactory:L0805 -> alvie:DFE252012F
- L11: value DFE252012F -> 600R; device alvie:DFE252012F -> GadgetFactory:L0805
- L13: value 10uH -> DFE252012F; device GadgetFactory:L0805 -> alvie:DFE252012F
- L14: value (none) -> 600R; device GadgetFactory:L0402 -> GadgetFactory:L0805
- L2: value DFE252012F -> 10uH; device alvie:DFE252012F -> GadgetFactory:L0805
- L3: value (none) -> 10uH
- L6: value 10uH -> (none)
- L8: value 10mH -> 10uH
- L9: value 600R -> 10uH
- Q11: value BSS84 -> 8MHz; device transistor-small-signal:BSS84 -> crystal:CRYSTALHC49U-V
- Q2, Q7: value 8MHz -> BSS84; device crystal:CRYSTALHC49U-V -> transistor-small-signal:BSS84
- Q4: value BSS123 -> 25MHz; device transistor-small-signal:BSS123 -> crystal:CRYSTALHC49U-V
- Q5: value 25MHz -> BSS84; device crystal:CRYSTALHC49U-V -> transistor-small-signal:BSS84
- Q6: value FDN338 -> 8MHz; device transistor-power:FDN360P -> crystal:CRYSTALHC49U-V
- Q8: value BSS84 -> BSS123; device transistor-small-signal:BSS84 -> transistor-small-signal:BSS123
- Q9: value BSS84 -> FDN338; device transistor-small-signal:BSS84 -> transistor-power:FDN360P
- R1: value 2K2 -> 470K
- R10, R38, R8, R9: value 10K -> 2K2
- R11, R36: value 20R -> 10K
- R13: value 0R/DNP -> 330R
- R14: value 100R -> 20R
- R15: value 100R -> 330R
- R16, R17: value 240K -> 330R
- R18: value 1K5/DNP -> 330R
- R19, R20, R21: value 20K -> 330R
- R22: value 6K2 -> 10K
- R23: value 100K -> 240K
- R24: value 20K -> 240K
- R25: value 100K -> 10K
- R27, R28, R32: value 100R -> 20K
- R29: value 100R -> 6K2
- R30: value 100R -> 12K1
- R31, R33: value 100R -> 100K
- R34: value 10K -> 20K
- R35: value 10K -> 2K2/DNP
- R37: value 20R -> 2K2/DNP
- R39: value 20R -> 49R9
- R4, R81: value 2K2 -> 10K
- R40: value 20R -> 0R
- R41: value 0R -> 49R9
- R42: value 0R -> 2K2
- R44: value 100K -> 49R9
- R46: value 2K2 -> 49R9
- R47, R79: value 2K2 -> 20R
- R48: value 2K2/DNP -> 20R
- R49: value 2K2/DNP -> 0R/DNP
- R5: value 6K2 -> 2K2
- R50, R62: value 10K -> 100R
- R51: value 1K5/DNP -> 100R
- R52: value 470K -> 10K
- R53: value 0R -> 1K5/DNP
- R54, R55: value 0R -> 330R
- R56, R61: value 0R/DNP -> 100R
- R57, R60: value 0R -> 100R
- R58, R59: value 330R -> 100R
- R63: value 10K -> 100K
- R64: value 10K -> 6K2
- R65, R66: value 10K -> 0R
- R67, R69: value 330R -> 0R
- R68, R70: value 330R -> 0R/DNP
- R7: value 240K -> 10K
- R71, R72: value 330R -> 1K5/DNP
- R73: value 330R -> 240K
- R74: value 330R -> 10K
- R75: value 56K -> 10K
- R76: value 0R -> 10K
- R77, R80: value 2K2 -> 1K5/DNP
- R78: value 10K -> 20R
- R82: value 12K1 -> 10K
- R83: value 49R9 -> 10K
- U$11: value STM32F030F4P6 -> PIN-1X8; device alvie:STM32F030F4P6 -> alvie:PIN-1X8
- U$12: value PIN-1X8 -> PIN-1X4; device alvie:PIN-1X8 -> alvie:PIN-1X4
- U$13: value PIN-1X8 -> PMS150C-U06; device alvie:PIN-1X8 -> alvie:PMS150C-U06
- U$14: value PN532_NFCB -> AP2000; device alvie:PN532_NFCB -> alvie:AP2000
- U$15: value STM32F070F6 -> MT3608; device alvie:STM32F070F6 -> alvie:MT3608
- U$16: value MIC550X -> PIN-1X10; device alvie:MIC550X -> alvie:PIN-1X10
- U$17: value PIN-1X4 -> PIN-1X10; device alvie:PIN-1X4 -> alvie:PIN-1X10
- U$25: value SR410361N -> PN532_NFCB; device alvie:SR410361N -> alvie:PN532_NFCB
- U$26: value PIN-1X8 -> PIN-1X10; device alvie:PIN-1X8 -> alvie:PIN-1X10
- U$27: value TSSOP16 -> PIN-1X10; device alvie:TSSOP16 -> alvie:PIN-1X10
- U$28: value PFS154-S16 -> MIC550X; device alvie:PFS154-S16 -> alvie:MIC550X
- U$29: value PIN-1X4 -> STM32F070F6; device alvie:PIN-1X4 -> alvie:STM32F070F6
- U$3: value MT3608 -> SR410361N; device alvie:MT3608 -> alvie:SR410361N
- U$30: value CC2530 -> PIN-1X4; device alvie:CC2530 -> alvie:PIN-1X4
- U$6: value PIN-1X4 -> PIN-1X8; device alvie:PIN-1X4 -> alvie:PIN-1X8
- U$7: value PIN-1X8 -> PFS154-S16; device alvie:PIN-1X8 -> alvie:PFS154-S16
- U$8: value PMS150C-U06 -> PIN-1X4; device alvie:PMS150C-U06 -> alvie:PIN-1X4
- U$9: value PFS154-S16 -> TSSOP16; device alvie:PFS154-S16 -> alvie:TSSOP16
- U1: value MIC550X -> STM32F107RCT6; device alvie:MIC550X -> ST Microelctronics_By_element14_Batch_1:STM32F107RCT6
- U2: value STM32F107RCT6 -> ESP-WROOM-32; device ST Microelctronics_By_element14_Batch_1:STM32F107RCT6 -> esp32:ESP-WROOM-32
- U3: value ESP-WROOM-32 -> MIC550X; device esp32:ESP-WROOM-32 -> alvie:MIC550X
- renumbered T2 to T1
Connections:
- removed net +3V3_CC: C75.2, C76.2, C77.2, C78.2, C79.2, C80.2, C81.2, C83.2, L16.2, R87A.1, U$30G$2.AVDD1, U$30G$2.AVDD2, U$30G$2.AVDD3, U$30G$2.AVDD4, U$30G$2.AVDD5, U$30G$2.AVDD6, U$30G$2.DVDD1, U$30G$2.DVDD2, U$31.4
- removed net CCLED1: R77A.2, U$30G$1.P1_0
- removed net CCLED2: R81A.2, U$30G$1.P1_1
- removed net CC_MISO: R76A.2, U$30G$1.P1_7
- removed net CC_MOSI: R42A.2, U$30G$1.P1_6
- removed net CC_SCK: R41A.2, U$30G$1.P1_5
- removed net DEBUG_C: U$30G$1.P2_2, U$31.2
- removed net DEBUG_D: U$30G$1.P2_1, U$31.3
- removed net N$106: C85.2, Q12.1, U$30G$1.P2_4/XOSC32K_Q1
- removed net N$79: C70.2, C73.2, L15.1
- removed net N$80: C71.1, U$30G$3.RF_P
- removed net N$82: C71.2, C72.2, L14.1
- removed net N$83: C73.1, C74.2, L14.2
- removed net N$84: C74.1, J7.1
- removed net N$85: R75A.2, U$30G$3.RBIAS
- removed net N$86: C82.2, U$30G$2.DCOUPL
- removed net N$87: LED8.C, R81A.1
- removed net N$88: C86.2, Q13.3, U$30G$3.XOSC_Q2
- removed net N$89: C87.2, Q13.1, U$30G$3.XOSC_Q1
- removed net N$90: C84.2, Q12.3, U$30G$1.P2_3/XOSC32K_Q2
- new net S0: U$16.1, X2-6.1
- new net S1: U$18.2, X2-7.1
- new net S10: U$18.5, X2-17.1
- new net S11: U$17.5, X2-18.1
- new net S12: U$16.5, X2-19.1
- new net S13: U$18.6, X2-20.1
- new net S14: U$17.6, X2-21.1
- new net S15: U$16.6, X2-22.1
- new net S16: U$18.7, X2-23.1
- new net S17: U$17.7, X2-24.1
- new net S18: U$16.7, X2-25.1
- new net S19: U$18.8, X2-26.1
- new net S2: U$17.2, X2-8.1
- new net S20: U$17.8, X2-27.1
- new net S21: U$16.8, X2-28.1
- new net S22: U$18.9, X2-30.1
- new net S23: U$17.9, X2-32.1
- new net S24: U$16.9, X2-34.1
- new net S25: U$18.10, X2-36.1
- new net S26: U$17.10, X2-38.1
- new net S27: U$16.10, X2-39.1
- new net S3: U$16.2, X2-9.1
- new net S4: U$18.3, X2-10.1
- new net S5: U$17.3, X2-12.1
- new net S6: U$16.3, X2-13.1
- new net S7: U$18.4, X2-14.1
- new net S8: U$17.4, X2-15.1
- new net S9: U$16.4, X2-16.1
- new net S_FB: R71A.1, R72A.2, U$14.FB
- new net S_SW: L9.2, U$14.SW
- new net S_VIN: C42.2, JP7.2, L9.1, U$14.SHDN, U$14.VIN
- new net S_VOUT: C54.2, C55.2, JP8.1, R71A.2, U$14.VOUT
- new net VCC3: C71.2, C74.2, IC8.VCC, IC9.VOUT, R77A.2, U$26.10, U$26.9
- new net VCCI: C67.2, IC9.EN, IC9.VIN, R77A.1, U$27.10, U$27.9
- new net X0: IC8.PB4, U$26.2
- new net X1: IC8.PB5, U$26.3
- new net X10: IC8.PB0, U$27.5
- new net X11: IC8.PA0, U$27.6
- new net X12: IC8.PA4, U$27.7
- new net X13: IC8.PA3, U$27.8
- new net X2: IC8.PB6, U$26.4
- new net X3: IC8.PB7, U$26.5
- new net X4: IC8.PA7, U$26.6
- new net X5: IC8.PA6, U$26.7
- new net X6: IC8.PA5, U$26.8
- new net X7: IC8.PB3, U$27.2
- new net X8: IC8.PB2, U$27.3
- new net X9: IC8.PB1, U$27.4
- net +15V: now also C13.1, C57.1, C58.2, C59.2, D2.C, IC2P.V+, R73A.2; no longer C11.1, C12.2, C13.2, C8.1, D3.C, IC1P.V+, R7A.2
- net +3V3: now also C1.1, C10.2, C11.2, C15.2, C16.2, C17.2, C2.1, C22.1, C24.1, C27.1, C3.1, C30.2, C38.2, C39.2, C4.1, C47.1, C49.1, C52.1, C62.2, C64.2, C65.2, C76.2, C77.2, C79.2, C8.2, C80.2, IC1.VDD1A, IC1.VDD2A, IC1.VDDIO, IC4.FB, J5.2, JP1.2, JP9.1, L1.1, L12.1, L13.2, M3.VOUT, Q1.S, Q2.S, Q5.S, Q7.S, R10A.2, R11A.2, R1A.1, R22A.2, R25A.2, R35A.2, R36A.2, R37A.2, R4A.2, R52A.2, R53A.2, R54A.2, R55A.2, R63A.1, R75A.2, R7A.2, R83A.2, R8A.2, U$10.4, U$19.VDD, U$22.2, U$23.7, U$25.VCC, U$28.VOUT, U$29.VDD, U$29.VDDA, U$30.1, U$7.VCC, U$8.1, U1.VBAT, U1.VDD_1, U1.VDD_2, U1.VDD_3, U1.VDD_4, U3.VOUT, X1-2.1, X1-3.1; no longer C14.2, C15.1, C18.1, C19.1, C2.2, C26.1, C28.1, C30.1, C36.2, C4.2, C41.1, C42.1, C43.1, C45.1, C46.2, C51.2, C53.2, C54.2, C56.2, C59.2, C60.2, C61.2, C93.2, C94.2, C95.2, C96.2, IC11.VDD1A, IC11.VDD2A, IC11.VDDIO, IC15.FB, J1.2, JP5.1, JP7.2, L10.1, L16.1, L7.2, L8.1, LED7.A, LED8.A, M2.VOUT, Q10.S, Q11.S, Q6.S, Q8.S, R18A.2, R34A.2, R3A.2, R43A.2, R44A.1, R48A.2, R49A.2, R51A.2, R52A.1, R58A.2, R59A.2, R63A.2, R64A.2, R65A.2, R66A.2, R78A.2, R79A.2, R9A.2, SV1.1, U$10.2, U$11.VDD, U$13.7, U$14.VCC, U$15.VDD, U$15.VDDA, U$16.VOUT, U$17.1, U$28.VCC, U$29.4, U$33.1, U$6.1, U1.VOUT, U2.VBAT, U2.VDD_1, U2.VDD_2, U2.VDD_3, U2.VDD_4
- net +5V: now also C40.2, L7.1, USB2USB.VUSB; no longer C24.2, L4.1, USB1USB.VUSB
- net +5V_FILT: now also C43.1, L7.2, Q10.S, R64A.2, U3.EN, U3.VIN; no longer C25.1, L4.2, Q1.S, R5A.2, U1.EN, U1.VIN
- net A_MISO: now also J6.1; no longer J5.1
- net A_MOSI: now also J6.4; no longer J5.4
- net A_RESET: now also J6.5; no longer J5.5
- net A_SCK: now also J6.3; no longer J5.3
- net BOOT0: now also R43A.2; no longer R10A.2
- net CA0: now also Q1.G, R7A.1, U$7.PA6; no longer Q8.G, R63A.1, U$28.PA6
- net CA1: now also Q2.G, R11A.1, U$7.PA7; no longer Q9.G, R64A.1, U$28.PA7
- net CA2: now also Q3.G, R22A.1, U$7.PB7; no longer Q10.G, R65A.1, U$28.PB7
- net CA3: now also Q5.G, R25A.1, U$7.PB6; no longer Q11.G, R66A.1, U$28.PB6
- net CC_RST: now also U1.PC8, X1-22.1; no longer R87A.2, U$30G$1.RESET_N, U2.PC8
- net CC_RX: now also U1.PC12, X1-17.1; no longer U$30G$1.P0_2, U2.PC12
- net CC_SS: now also U1.PC9, X1-21.1; no longer U$30G$1.P1_4, U2.PC9
- net CC_TX: now also U1.PD2, X1-18.1; no longer U$30G$1.P0_3, U2.PD2
- net ESP_EN: now also U1.PA14, U2.EN; no longer U2.PA14, U3.EN
- net ESP_IO0: now also U1.PB10, U2.IO0; no longer U2.PB10, U3.IO0
- net ESP_MISO: now also R67A.2, R68A.2, U2.IO19; no longer R56A.2, R57A.2, R76A.1, U3.IO19
- net ESP_MOSI: now also R69A.2, R70A.2, U2.IO23; no longer R42A.1, R60A.2, R61A.2, U3.IO23
- net ESP_ON: now also Q9.G, R63A.2; no longer Q6.G, R44A.2
- net ESP_RX: now also U1.PC10, U2.RXD0; no longer U2.PC10, U3.RXD0
- net ESP_SCK: now also R66A.2, U2.IO18; no longer R41A.1, R55A.2, U3.IO18
- net ESP_TX: now also U1.PC11, U2.TXD0; no longer U2.PC11, U3.TXD0
- net ESP_VCC: now also Q9.D, U2.3V3; no longer Q6.D, U3.3V3
- net GND: now also C1.2, C11.1, C15.1, C18.1, C19.1, C2.2, C21.1, C24.2, C28.1, C29.1, C3.2, C30.1, C31.1, C34.2, C35.2, C4.2, C40.1, C41.1, C42.1, C45.1, C47.2, C49.2, C5.1, C52.2, C53.2, C56.2, C58.1, C60.2, C62.1, C64.1, C66.2, C70.2, C71.1, C73.2, C74.1, C75.2, C8.1, D4.K, IC1.VSS, IC4.AGND, IC4.MODE, IC4.PGND, IC5.12, IC6P.GND, IC6P.VEE, IC7P.GND, IC7P.VEE, IC8.GND, IC9.GND, J1.2, J3.1, J4.2, J6.6, JP10.1, JP11.1, JP4.1, JP5.2, JP7.1, JP8.2, Q8.S, R23A.1, R27A.1, R29A.1, R30A.1, R32A.1, R34A.1, R3A.2, R43A.1, R72A.1, R74A.1, R76A.1, S1.1, S2.2, U$12.3, U$12.4, U$13.GND, U$15.GND, U$18.1, U$19.VSS, U$20.GND, U$22.1, U$23.8, U$25.GND, U$26.1, U$27.1, U$29.VSS, U$30.4, U$7.GND, U$8.4, U1.VSSA, U1.VSS_1, U1.VSS_2, U1.VSS_3, U1.VSS_4, U2.GND, U2.GND@1, U2.GND@15, U2.GND@38, X1-11.1, X1-29.1, X1-31.1, X1-33.1, X1-35.1, X1-37.1, X1-4.1, X1-40.1, X1-5.1, X2-11.1, X2-29.1, X2-31.1, X2-33.1, X2-35.1, X2-37.1, X2-4.1, X2-40.1, X2-5.1; no longer C1.1, C11.2, C13.1, C15.2, C18.2, C19.2, C2.1, C21.2, C24.1, C28.2, C29.2, C3.1, C30.2, C31.2, C34.1, C35.1, C4.1, C40.2, C41.2, C42.2, C45.2, C47.1, C49.1, C52.1, C53.1, C56.1, C58.2, C60.1, C62.2, C63.2, C64.2, C66.1, C75.1, C83.1, C84.1, C85.1, C86.1, C87.1, C93.1, C94.1, C95.1, C96.1, C97.1, C98.1, C99.1, D2.K, IC11.VSS, IC15.AGND, IC15.MODE, IC15.PGND, IC2.12, IC4P.GND, IC4P.VEE, IC5P.GND, IC5P.VEE, J3.2, J4.1, J5.6, J6.2, J7.2, JP1.1, JP11.2, JP6.1, JP9.1, L15.2, Q12.2, Q12.4, Q13.2, Q13.4, Q4.S, R10A.1, R16A.1, R17A.1, R20A.1, R22A.1, R26A.1, R35A.1, R38A.1, R50A.2, R75A.1, R8A.1, S1.2, S2.1, SV1.3, SV1.4, U$11.VSS, U$13.8, U$15.VSS, U$16.GND, U$17.4, U$29.1, U$3.GND, U$30G$2.GND, U$30G$2.GND@1, U$30G$2.GND@2, U$30G$2.GND@3, U$30G$2.PAD, U$31.1, U$32.1, U$6.4, U$8.GND, U$9.GND, U1.GND, U2.VSSA, U2.VSS_1, U2.VSS_2, U2.VSS_3, U2.VSS_4, U3.GND@1, U3.GND@15, U3.GND@38
- net LCLK: now also U$10.2, U$7.PA0; no longer U$28.PA0, U$29.2
- net LDAT: now also U$10.3, U$7.PB0; no longer U$28.PB0, U$29.3
- net LED0: now also R2A.2; no longer R1A.2
- net LED1: now also R5A.2; no longer R2A.2
- net LED2: now also R9A.2; no longer R4A.2
- net MCO: now also R40A.1, U1.PA8; no longer R53A.1, U2.PA8
- net MCU_MISO: now also IC5.7, R59A.1, R60A.1, U$13.PA6, U$20.PA6; no longer IC2.7, R30A.1, R31A.1, U$8.PA6, U$9.PA6
- net MCU_MOSI: now also IC5.10, R61A.1, R62A.1, U$13.PA4, U$20.PA4; no longer IC2.10, R32A.1, R33A.1, U$8.PA4, U$9.PA4
- net MCU_PA0: now also IC5.11, R56A.1, U$20.PA0; no longer IC2.11, R27A.1, U$9.PA0
- net MCU_PA7: now also IC5.6, R57A.1, U$20.PA7; no longer IC2.6, R28A.1, U$9.PA7
- net MCU_SCK: now also IC5.9, R58A.1, U$13.PA3, U$20.PA3; no longer IC2.9, R29A.1, U$8.PA3, U$9.PA3
- net MISO: now also R59A.2, R62A.2; no longer R30A.2, R33A.2
- net MOSI: now also R60A.2, R61A.2; no longer R31A.2, R32A.2
- net N$1: now also R5A.1; no longer R2A.1
- net N$10: now also C45.2, C46.2, L11.1, U$19.VDDA; no longer C34.2, C35.2, L7.1, U$11.VDDA
- net N$100: now also IC3.13, U$11.5, U$9.12; no longer IC6.13, U$26.5, U$27.12
- net N$101: now also IC3.14, U$11.6, U$9.11; no longer IC6.14, U$26.6, U$27.11
- net N$102: now also IC3.12, U$11.4, U$9.13; no longer IC6.12, U$26.4, U$27.13
- net N$103: now also IC3.11, U$11.3, U$9.14; no longer IC6.11, U$26.3, U$27.14
- net N$104: now also IC3.10, U$11.2, U$9.15; no longer IC6.10, U$26.2, U$27.15
- net N$105: now also IC3.9, U$11.1, U$9.16; no longer IC6.9, U$26.1, U$27.16
- net N$11: now also C36.2, JP6.1, L6.2; no longer C20.2, JP4.1, L3.2
- net N$13: now also C41.2, J4.1, J5.1, L8.1; no longer C32.2, J2.1, J3.1, L6.1
- net N$14: now also C37.2, JP6.2; no longer C23.2, JP4.2
- net N$15: now also L6.1, Q7.D, Q8.D; no longer L3.1, Q3.D, Q4.D
- net N$16: now also L8.2, M3.SW; no longer L6.2, M2.SW
- net N$17: now also L14.1; no longer L12.1
- net N$18: now also Q7.G, R49A.1, R50A.1; no longer Q3.G, R13A.1, R14A.1
- net N$19: now also Q8.G, R51A.1; no longer Q4.G, R15A.1
- net N$2: now also C44.2, L10.1, Q10.D, U$15.EN, U$15.IN; no longer C6.2, L2.1, Q1.D, U$3.EN, U$3.IN
- net N$20: now also R12A.1, USB1USB.D-; no longer R39A.1, USB2USB.D-
- net N$21: now also R2A.1; no longer R1A.1
- net N$22: now also R14A.1, USB1USB.D+; no longer R40A.1, USB2USB.D+
- net N$23: now also JP9.2, R76A.2, U$19.BOOT0; no longer JP5.2, R35A.2, U$11.BOOT0
- net N$24: now also U$12.1, X2-1.1; no longer LED7.C, R77A.1
- net N$25: now also R65A.2, U2.IO5; no longer R54A.2, U3.IO5
- net N$26: now also R38A.1; no longer R45A.1
- net N$27: now also R42A.1; no longer R46A.1
- net N$28: now also R45A.1; no longer R47A.1
- net N$29: now also R78A.1; no longer R36A.1
- net N$3: now also R9A.1; no longer R4A.1
- net N$30: now also IC5.16; no longer IC2.16
- net N$31: now also IC5.15; no longer IC2.15
- net N$32: now also IC5.14; no longer IC2.14
- net N$33: now also R79A.1; no longer R37A.1
- net N$34: now also IC6A.X, IC7A.X; no longer IC4A.X, IC5A.X
- net N$35: now also IC5.13; no longer IC2.13
- net N$36: now also R47A.1, USB2USB.D-; no longer R11A.1, USB1USB.D-
- net N$37: now also R48A.1, USB2USB.D+; no longer R12A.1, USB1USB.D+
- net N$38: now also IC6A.X7, JP12.1; no longer IC4A.X7, JP8.1
- net N$39: now also L4.1, USB1USB.VUSB; no longer L9.1, USB2USB.VUSB
- net N$4: now also L2.2; no longer L1.2
- net N$40: now also IC1.RBIAS, R30A.2; no longer IC11.RBIAS, R82A.2
- net N$41: now also C6.2, J1.1, L3.1; no longer C66.2, J6.1, L13.1
- net N$42: now also R73A.1, R74A.2, U$15.FB; no longer R7A.1, R8A.2, U$3.FB
- net N$43: now also C63.2, D3.K, D4.A; no longer C5.2, D1.K, D2.A
- net N$44: now also C35.1; no longer C57.1
- net N$45: now also C34.1; no longer C58.1
- net N$46: now also R54A.1; no longer R58A.1
- net N$47: now also L3.2, M2.SW; no longer L13.2, M3.SW
- net N$48: now also C18.2, JP5.1, M2.VOUT; no longer C67.2, JP11.1, M3.VOUT
- net N$49: now also IC7A.X0, JP13.8; no longer IC5A.X0, JP10.8
- net N$5: now also C5.2, J2.1, JP3.2, L2.1; no longer C1.2, J1.1, JP2.2, L1.1
- net N$50: now also IC2B.-IN, R28A.2, R29A.2; no longer IC1B.-IN, R21A.2, R22A.2
- net N$51: now also IC2A.-IN, R26A.2, R27A.2; no longer IC1A.-IN, R19A.2, R20A.2
- net N$52: now also IC6A.X0, JP12.8; no longer IC4A.X0, JP8.8
- net N$53: now also R55A.1; no longer R59A.1
- net N$54: now also IC5.1; no longer IC2.1
- net N$55: now also IC5.2; no longer IC2.2
- net N$56: now also C28.2, L5.2, R39A.2, R41A.2, R44A.2, R46A.2; no longer C99.2, L10.2, R83A.2, R84A.2, R85A.2, R86A.2
- net N$57: now also IC5.3; no longer IC2.3
- net N$58: now also C21.2, C23.2, IC1.VDDCR; no longer C97.2, C98.2, IC11.VDDCR
- net N$59: now also IC5.4; no longer IC2.4
- net N$60: now also IC6A.X1, JP12.7; no longer IC4A.X1, JP8.7
- net N$61: now also IC6A.X3, JP12.5; no longer IC4A.X3, JP8.5
- net N$62: now also IC6A.X4, JP12.4; no longer IC4A.X4, JP8.4
- net N$63: now also IC6A.X5, JP12.3; no longer IC4A.X5, JP8.3
- net N$64: now also IC6A.X6, JP12.2; no longer IC4A.X6, JP8.2
- net N$65: now also Q2.D, U$3.CA1; no longer Q9.D, U$25.CA1
- net N$66: now also J6.2; no longer J5.2
- net N$67: now also IC7A.X1, JP13.7; no longer IC5A.X1, JP10.7
- net N$68: now also IC7A.X2, JP13.6; no longer IC5A.X2, JP10.6
- net N$69: now also IC7A.X3, JP13.5; no longer IC5A.X3, JP10.5
- net N$7: now also C14.2; no longer C3.2
- net N$70: now also IC6A.X2, JP12.6; no longer IC4A.X2, JP8.6
- net N$71: now also IC7A.X4, JP13.4; no longer IC5A.X4, JP10.4
- net N$72: now also IC7A.X5, JP13.3; no longer IC5A.X5, JP10.3
- net N$73: now also IC7A.X6, JP13.2; no longer IC5A.X6, JP10.2
- net N$74: now also IC7A.X7, JP13.1; no longer IC5A.X7, JP10.1
- net N$75: now also Q3.D, U$3.CA2; no longer Q10.D, U$25.CA2
- net N$76: now also Q1.D, U$3.CA0; no longer Q8.D, U$25.CA0
- net N$77: now also Q5.D, U$3.CA3; no longer Q11.D, U$25.CA3
- net N$78: now also U$12.2, U$17.1, X2-2.1, X2-3.1; no longer C70.1, U$30G$3.RF_N
- net N$8: now also C29.2, R36A.1, U$8.2; no longer C10.2, R9A.1, U$6.2
- net N$81: now also IC3.8, U$6.1, U$9.1; no longer IC6.8, U$27.1, U$7.1
- net N$91: now also IC3.7, U$6.2, U$9.2; no longer IC6.7, U$27.2, U$7.2
- net N$92: now also IC3.6, U$6.3, U$9.3; no longer IC6.6, U$27.3, U$7.3
- net N$93: now also IC3.5, U$6.4, U$9.4; no longer IC6.5, U$27.4, U$7.4
- net N$94: now also IC3.4, U$6.5, U$9.5; no longer IC6.4, U$27.5, U$7.5
- net N$95: now also IC3.3, U$6.6, U$9.6; no longer IC6.3, U$27.6, U$7.6
- net N$96: now also IC3.2, U$6.7, U$9.7; no longer IC6.2, U$27.7, U$7.7
- net N$97: now also IC3.1, U$6.8, U$9.8; no longer IC6.1, U$27.8, U$7.8
- net N$98: now also IC3.16, U$11.8, U$9.9; no longer IC6.16, U$26.8, U$27.9
- net N$99: now also IC3.15, U$11.7, U$9.10; no longer IC6.15, U$26.7, U$27.10
- net NBOOT0: now also R82A.2, U$29.BOOT0; no longer R38A.2, U$15.BOOT0
- net NIRQ: now also U$25.IRQ, U$29.PA1; no longer U$14.IRQ, U$15.PA1
- net NLED0: now also R38A.2, U1.PA13; no longer R45A.2, U2.PA13
- net NLED1: now also R42A.2, U1.PB14; no longer R46A.2, U2.PB14
- net NLED2: now also R45A.2, U1.PB15; no longer R47A.2, U2.PB15
- net NNRST: now also R83A.1, U$29.NRST; no longer R43A.1, U$15.NRST
- net NOSC_IN: now also C81.2, Q11.2, U$29.PF0/OSC_IN; no longer C47.2, Q7.2, U$15.PF0/OSC_IN
- net NOSC_OUT: now also C82.2, Q11.1, U$29.PF1/OSC_OUT; no longer C52.2, Q7.1, U$15.PF1/OSC_OUT
- net NRST: now also R52A.1, S2.1; no longer R6A.1, S1.1
- net NRSTO: now also U$25.RSTO, U$29.PA0; no longer U$14.RSTO, U$15.PA0
- net NSWCLK: now also U$29.PA14, U$30.3; no longer U$15.PA14, U$17.3
- net NSWDIO: now also U$29.PA13, U$30.2; no longer U$15.PA13, U$17.2
- net NUSBDM: now also R78A.2, U$29.PA9/PA11; no longer R36A.2, U$15.PA9/PA11
- net NUSBDP: now also R79A.2, R80A.1, U$29.PA10/PA12; no longer R37A.2, R51A.1, U$15.PA10/PA12
- net N_MISO: now also U$25.MISO, U$29.PA6; no longer U$14.MISO, U$15.PA6
- net N_MOSI: now also U$25.MOSI, U$29.PA7; no longer U$14.MOSI, U$15.PA7
- net N_RX: now also U$25.SDA/TX, U$29.PA3; no longer U$14.SDA/TX, U$15.PA3
- net N_SCK: now also U$25.SCK, U$29.PA5; no longer U$14.SCK, U$15.PA5
- net N_SS: now also U$25.SS, U$29.PA4; no longer U$14.SS, U$15.PA4
- net N_TX: now also U$25.SCL/RX, U$29.PA2; no longer U$14.SCL/RX, U$15.PA2
- net OSC_IN: now also C31.2, Q6.2; no longer C16.2, Q2.2
- net OSC_OUT: now also C32.2, Q6.1; no longer C17.2, Q2.1
- net PA0: now also U$19.PA0, U$23.3; no longer U$11.PA0, U$13.3
- net PA1: now also U$19.PA1, U$23.2; no longer U$11.PA1, U$13.2
- net PA10: now also U$19.PA10; no longer U$11.PA10
- net PA13: now also U$19.PA13/SWDIO, U$21.2; no longer U$11.PA13/SWDIO, U$12.2
- net PA14: now also U$19.PA14/SWCLK, U$21.1; no longer U$11.PA14/SWCLK, U$12.1
- net PA15/NSS: now also R65A.1, U1.PA15; no longer R54A.1, U2.PA15
- net PA2: now also U$19.PA2, U$23.1; no longer U$11.PA2, U$13.1
- net PA3: now also U$19.PA3, U$21.8; no longer U$11.PA3, U$12.8
- net PA3/ADC3: now also U1.PA3, X1-30.1; no longer U$33.2, U2.PA3
- net PA4: now also U$19.PA4, U$21.7; no longer U$11.PA4, U$12.7
- net PA4/DAC1: now also U1.PA4, X1-32.1; no longer U$33.3, U2.PA4
- net PA5: now also U$19.PA5, U$21.6; no longer U$11.PA5, U$12.6
- net PA5/DAC2: now also U1.PA5, X1-34.1; no longer U$32.3, U2.PA5
- net PA6: now also U$19.PA6, U$21.5; no longer U$11.PA6, U$12.5
- net PA7: now also U$19.PA7, U$21.4; no longer U$11.PA7, U$12.4
- net PA9: now also U$19.PA9; no longer U$11.PA9
- net PB1: now also U$19.PB1, U$21.3; no longer U$11.PB1, U$12.3
- net PB6/UART1_TX: now also U1.PB6, X1-12.1; no longer SV1.24, U2.PB6
- net PB7/UART1_RX: now also U1.PB7, X1-13.1; no longer SV1.23, U2.PB7
- net PEDAL: now also JP11.2, R81A.1; no longer JP9.2, R62A.1
- net PF0: now also U$19.PF0/OSC_IN, U$23.6; no longer U$11.PF0/OSC_IN, U$13.6
- net PF1: now also U$19.PF1/OSC_OUT, U$23.5; no longer U$11.PF1/OSC_OUT, U$13.5
- net PHY_LED0: now also IC1.LED1/REGOFF; no longer IC11.LED1/REGOFF
- net PHY_LED1: now also IC1.LED2/NINTSEL; no longer IC11.LED2/NINTSEL
- net PWM1: now also R50A.2, R51A.2; no longer R14A.2, R15A.2
- net PWM2: now also R49A.2; no longer R13A.2
- net PWRON: now also Q10.G, R64A.1; no longer Q1.G, R5A.1
- net REG33IN: now also C51.2, D1.C, IC4.AVIN, IC4.EN, IC4.PVIN, J3.3, X1-1.1; no longer C49.2, D4.C, IC15.AVIN, IC15.EN, IC15.PVIN, J4.3, SV1.2
- net RMII_CRS_DV: now also IC1.CRS_DV/MODE2, U1.PA7; no longer IC11.CRS_DV/MODE2, U2.PA7
- net RMII_MDC: now also IC1.MDC, R8A.1, U1.PC1; no longer IC11.MDC, R79A.1, U2.PC1
- net RMII_MDIO: now also IC1.MDIO, R10A.1, U1.PA2; no longer IC11.MDIO, R80A.1, U2.PA2
- net RMII_NRST: now also IC1.NRST, R4A.1, U1.PA6; no longer IC11.NRST, R78A.1, U2.PA6
- net RMII_REF_CLK: now also IC1.NINT/REFCLK0, U1.PA1; no longer IC11.NINT/REFCLK0, U2.PA1
- net RMII_RXD0: now also IC1.RXD0/MODE0, U1.PC4; no longer IC11.RXD0/MODE0, U2.PC4
- net RMII_RXD1: now also IC1.RXD1/MODE1, U1.PC5; no longer IC11.RXD1/MODE1, U2.PC5
- net RMII_TXD0: now also IC1.TXD0, U1.PB12; no longer IC11.TXD0, U2.PB12
- net RMII_TXD1: now also IC1.TXD1, U1.PB13; no longer IC11.TXD1, U2.PB13
- net RMII_TX_EN: now also IC1.TXEN, U1.PB11; no longer IC11.TXEN, U2.PB11
- net RX: now also JP4.2; no longer JP3.2
- net RXM1: now also IC1.TXN, R41A.1; no longer IC11.TXN, R84A.1
- net RXP1: now also IC1.TXP, R39A.1; no longer IC11.TXP, R83A.1
- net SA: now also R13A.2, U$3.A; no longer R67A.2, U$25.A
- net SB: now also R15A.2, U$3.B; no longer R68A.2, U$25.B
- net SC: now also R16A.2, U$3.C; no longer R69A.2, U$25.C
- net SCK: now also R58A.2; no longer R29A.2
- net SD: now also R17A.2, U$3.D; no longer R70A.2, U$25.D
- net SDP: now also R21A.2, U$3.DP; no longer R74A.2, U$25.DP
- net SE: now also R18A.2, U$3.E; no longer R71A.2, U$25.E
- net SEG_A: now also R13A.1, U$7.PA3; no longer R67A.1, U$28.PA3
- net SEG_B: now also R15A.1, U$7.PB1; no longer R68A.1, U$28.PB1
- net SEG_C: now also R16A.1, U$7.PB5; no longer R69A.1, U$28.PB5
- net SEG_D: now also R17A.1, U$7.PB2; no longer R70A.1, U$28.PB2
- net SEG_DP: now also R21A.1, U$7.PB3; no longer R74A.1, U$28.PB3
- net SEG_E: now also R18A.1, U$7.PA4; no longer R71A.1, U$28.PA4
- net SEG_F: now also R19A.1, U$7.PA5; no longer R72A.1, U$28.PA5
- net SEG_G: now also R20A.1, U$7.PB4; no longer R73A.1, U$28.PB4
- net SEL_A0: now also IC7A.A; no longer IC5A.A
- net SEL_A1: now also IC6A.A; no longer IC4A.A
- net SEL_B0: now also IC7A.B; no longer IC5A.B
- net SEL_B1: now also IC6A.B; no longer IC4A.B
- net SEL_C0: now also IC7A.C; no longer IC5A.C
- net SEL_C1: now also IC6A.C; no longer IC4A.C
- net SEL_INH: now also IC6A.INH, IC7A.INH; no longer IC4A.INH, IC5A.INH
- net SF: now also R19A.2, U$3.F; no longer R72A.2, U$25.F
- net SG: now also R20A.2, U$3.G; no longer R73A.2, U$25.G
- net STM_PA0: now also R56A.2; no longer R27A.2
- net STM_PA7: now also R57A.2; no longer R28A.2
- net SW: now also JP2.2, R6A.1; no longer JP1.2, R3A.1
- net SWIM: now also U$8.3; no longer U$6.3
- net TX: now also JP4.3; no longer JP3.3
- net TXM1: now also IC1.RXN, R46A.1; no longer IC11.RXN, R86A.1
- net TXP1: now also IC1.RXP, R44A.1; no longer IC11.RXP, R85A.1
- net UART1RX: now also U1.PA10, X1-19.1; no longer SV1.18, U2.PA10
- net UART1TX: now also U1.PA9, X1-20.1; no longer SV1.17, U2.PA9
- net USBDM: now also R47A.2; no longer R11A.2
- net USBDP: now also R48A.2, R53A.1; no longer R12A.2, R18A.1
- net USBPWR: now also D1.A, L4.2; no longer D4.A, L9.2
- net USBPWR1: now also C78.2, L14.2, U$28.EN, U$28.VIN; no longer C55.2, L12.2, U$16.EN, U$16.VIN
- net VDDA: now also C56.1, L12.2; no longer C31.1, L5.2
- net VDD_OUT: now also C25.1, C53.1, IC2A.OUT, IC5.5, R26A.1, R33A.2, U$13.VCC, U$20.VCC; no longer C21.1, C27.1, IC1A.OUT, IC2.5, R19A.1, R25A.2, U$8.VCC, U$9.VCC
- net VDD_PWM: now also IC2A.+IN, R23A.2; no longer IC1A.+IN, R16A.2
- net VDD_SENS: now also R33A.1, R34A.2; no longer R25A.1, R26A.2
- net VEE: now also C13.2, C66.1, D3.A, IC2P.V-; no longer C7.1, C8.2, D1.A, IC1P.V-
- net VNEG_PWM: now also C63.1; no longer C5.1
- net VPP_OUT: now also C26.1, C60.1, IC2B.OUT, IC5.8, R28A.1, R31A.2, U$13.PA5, U$20.PA5; no longer C22.1, C29.1, IC1B.OUT, IC2.8, R21A.1, R23A.2, U$8.PA5, U$9.PA5
- net VPP_PWM: now also IC2B.+IN, R24A.2; no longer IC1B.+IN, R17A.2
- net VPP_SENS: now also R31A.1, R32A.2; no longer R23A.1, R24A.2
- net VSW: now also D2.A, L10.2, U$15.SW; no longer D3.A, L2.2, U$3.SW
- net V_BATT: now also C70.1, C72.2, C73.1, C75.1, IC6P.VCC, IC7P.VCC, JP10.2, R81A.2; no longer C62.1, C63.1, C64.1, C65.2, IC4P.VCC, IC5P.VCC, JP6.2, R62A.2
- net XBOOT0: now also JP1.1, R3A.1, U1.BOOT0; no longer JP7.1, R50A.1, U2.BOOT0
- net XI: now also IC1.XTAL1/CLKIN, R40A.2; no longer IC11.XTAL1/CLKIN, R53A.2
- net XNRST: now also C61.2, R75A.1, U$19.NRST, U$23.4; no longer C37.2, R34A.1, U$11.NRST, U$13.4
- net XOSC_IN: now also C19.2, Q4.2, U1.PD0_OSC_IN; no longer C38.2, Q5.2, U2.PD0_OSC_IN
- net XOSC_OUT: now also C20.2, Q4.1, U1.PD1_OSC_OUT; no longer C39.2, Q5.1, U2.PD1_OSC_OUT
- net XPA0: now also U1.PA0-WKUP, X1-28.1; no longer SV1.12, U2.PA0-WKUP
- net XPB0/ADC8: now also U1.PB0, X1-36.1; no longer U$32.2, U2.PB0
- net XPB1: now also U1.PB1, X1-38.1; no longer U$33.4, U2.PB1
- net XPB2: now also U1.PB2, X1-39.1; no longer U$32.4, U2.PB2
- net XPC0: now also U1.PC0, X1-25.1; no longer SV1.13, U2.PC0
- net XPC13: now also U1.PC13-TAMPER-RTC, X1-14.1; no longer SV1.22, U2.PC13-TAMPER-RTC
- net XPC14: now also U1.PC14-OSC32_IN, X1-15.1; no longer SV1.19, U2.PC14-OSC32_IN
- net XPC15: now also U1.PC15-OSC32_OUT, X1-16.1; no longer SV1.20, U2.PC15-OSC32_OUT
- net XPC2: now also U1.PC2, X1-26.1; no longer SV1.14, U2.PC2
- net XPC3: now also U1.PC3, X1-27.1; no longer SV1.11, U2.PC3
- net XPC6: now also U1.PC6, X1-24.1; no longer SV1.15, U2.PC6
- net XPC7: now also U1.PC7, X1-23.1; no longer SV1.16, U2.PC7
- net XSCL: now also R35A.1, U$22.3, U1.PB8, X1-6.1; no longer R48A.1, SV1.26, U$10.3, U2.PB8
- net XSDA: now also R37A.1, U$22.4, U1.PB9, X1-7.1; no longer R49A.1, SV1.25, U$10.4, U2.PB9
- net XSPI_MISO: now also R67A.1, R70A.1, U1.PB4, X1-9.1; no longer R57A.1, R61A.1, U2.PB4
- net XSPI_MOSI: now also R68A.1, R69A.1, U1.PB5, X1-10.1; no longer R56A.1, R60A.1, U2.PB5
- net XSPI_SCK: now also R66A.1, U1.PB3, X1-8.1; no longer R55A.1, U2.PB3
- net XSW: now also IC4.SW, L13.1; no longer IC15.SW, L11.1
- net XUSBDM: now also R12A.2, U1.PA11; no longer R39A.2, U2.PA11
- net XUSBDP: now also R14A.2, U1.PA12; no longer R40A.2, U2.PA12
- net XVDDA: now also C12.2, C7.1, L1.2, U1.VDDA; no longer C40.1, C44.2, L8.2, U2.VDDA
- net XXNRST: now also R1A.2, S1.2, U1.NRST; no longer R52A.2, S2.2, U2.NRST
Other:
- note removed: "pa_ce"
- note removed: "pa_tx_rx"
- moved on the sheet: C1, C10, C11, C12, C13, C14, C15, C16, C17, C18, C19, C2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

Commit message: Production
Parts:
- C39, C67: value (none) -> 22uF
- C42, C55, C72: value (none) -> 10uF
- C70, C73, C75: value (none) -> 100nF
- L1: value 10mH -> 10uH
- L6: value (none) -> 150nH
Other:
- note added: "ALD192/1-1"
- note added: "ALD192/10-1"
- note added: "ALD192/2-1"
- note added: "ALD192/3-1"
- note added: "ALD192/4-1"
- note added: "ALD192/5-1"
- note added: "ALD192/6-1"
- note added: "ALD192/7-1"
- note added: "ALD192/8-1"
- note added: "ALD192/9-1"
- note added: "AUDIO player"
- note added: "Attiny switch"
- note added: "Battery-powered STM32030"
- note added: "ETH Bridge"
- note added: "LCD Display"
- note added: "NFC USBizer"
- note added: "PADAUK Programmer"
- note added: "PADAUK breakout"
- note added: "SOIC16/TSSOP16 Addaptor"
- note added: "STEP UP Adjustable"
- moved on the sheet: IC3, U$11, U$6, U$9
